File: Micromouse/MPU6500.kicad_sch (KiCad schematic)
At the start: 5 parts, among them U5 LSM6DSRTR

Commit message: Añadiendo el chasis de minisumo
Parts:
- removed R21, R22: 10k, Resistor_SMD:R_0201_0603Metric, symbol Device:R
Connections:
- net SDA renamed MOSI
- net SDO/SA0 renamed MISO
