File: Micromouse/AS5048_Der.kicad_sch (KiCad schematic)
At the start: 6 parts, among them J10 AS5048_Der, U4 AS5048B-HTSP

Commit message: Añadiendo el chasis de minisumo
Connections:
- net +3V0_s: now also U4.4 (A1)
- net GND_s: now also U4.6 (TEST_6); no longer U4.4 (A1)
- no-connect marks 6 -> 5
Changed lines of the file:
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@@
 	)
 	(junction
-		(at 121.92 92.075)
+		(at 123.825 104.775)
 		(diameter 0)
 		(color 0 0 0 0)
@@
 	)
 	(no_connect
-		(at 125.73 107.315)
-	)
-	(no_connect
 		(at 161.29 94.615)
 	)
@@
 	(wire
 		(pts
-			(xy 121.92 92.075) (xy 125.73 92.075)
+			(xy 125.73 107.315) (xy 123.825 107.315)
+		)
+		(stroke
+			(width 0)
+			(type default)
+		)
+	)
+	(wire
+		(pts
+			(xy 123.825 104.775) (xy 125.73 104.775)
+		)
+		(stroke
+			(width 0)
+			(type default)
+		)
+	)
+	(wire
+		(pts
+			(xy 123.825 107.315) (xy 123.825 104.775)
 		)
 		(stroke
@@
 	(wire
 		(pts
-			(xy 118.11 92.075) (xy 121.92 92.075)
-		)
-		(stroke
-			(width 0)
-			(type default)
-		)
-	)
-	(wire
-		(pts
-			(xy 125.73 89.535) (xy 121.92 89.535)
+			(xy 118.11 92.075) (xy 125.73 92.075)
 		)
 		(stroke
@@
 	(wire
 		(pts
+			(xy 118.11 89.535) (xy 125.73 89.535)
+		)
+		(stroke
+			(width 0)
+			(type default)
+		)
+	)
+	(wire
+		(pts
 			(xy 84.455 92.075) (xy 86.995 92.075)
 		)
@@
 	(wire
 		(pts
-			(xy 118.11 104.775) (xy 125.73 104.775)
+			(xy 118.11 104.775) (xy 123.825 104.775)
 		)
 		(stroke
@@
 		(pts
 			(xy 114.935 97.155) (xy 125.73 97.155)
-		)
-		(stroke
-			(width 0)
-			(type default)
-		)
-	)
-	(wire
-		(pts
-			(xy 121.92 89.535) (xy 121.92 92.075)
 		)
 		(stroke
@@
 		)
 	)
+	(label "+3V0_s"
+		(at 118.11 89.535 180)
+		(effects
+			(font
+				(size 1.27 1.27)
+			)
+			(justify right bottom)
+		)
+	)

Commit message: Commit de prueba
Parts:
- J10: footprint (none) -> MicromouseHuellas:Encoder1
- renumbered C25 to C47, C26 to C48, R19 to R33, R20 to R34
Changed lines of the file:
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@@
 		(on_board yes)
 		(dnp no)
-		(property "Reference" "R20"
+		(property "Reference" "R34"
 			(at 107.95 101.6 90)
 			(effects
@@
 			(project "Half-Size Micromouse"
 				(path "/96b72c82-8e98-4b00-820e-849de0fa96c7/358c7740-1065-4f93-94de-62d9b382bca9"
-					(reference "R20")
+					(reference "R34")
 					(unit 1)
 				)
@@
 		(on_board yes)
 		(dnp no)
-		(property "Reference" "R19"
+		(property "Reference" "R33"
 			(at 107.95 95.25 90)
 			(effects
@@
 			(project "Half-Size Micromouse"
 				(path "/96b72c82-8e98-4b00-820e-849de0fa96c7/358c7740-1065-4f93-94de-62d9b382bca9"
-					(reference "R19")
+					(reference "R33")
 					(unit 1)
 				)
@@
 		(on_board yes)
 		(dnp no)
-		(property "Reference" "C25"
+		(property "Reference" "C47"
 			(at 187.325 88.265 0)
 			(effects
@@
 			(project "Half-Size Micromouse"
 				(path "/96b72c82-8e98-4b00-820e-849de0fa96c7/358c7740-1065-4f93-94de-62d9b382bca9"
-					(reference "C25")
+					(reference "C47")
 					(unit 1)
 				)
@@
 			)
 		)
-		(property "Footprint" ""
+		(property "Footprint" "MicromouseHuellas:Encoder1"
 			(at 79.375 92.075 0)
 			(effects
@@
 		(on_board yes)
 		(dnp no)
-		(property "Reference" "C26"
+		(property "Reference" "C48"
 			(at 199.39 88.265 0)
 			(effects
@@
 			(project "Half-Size Micromouse"
 				(path "/96b72c82-8e98-4b00-820e-849de0fa96c7/358c7740-1065-4f93-94de-62d9b382bca9"
-					(reference "C26")
+					(reference "C48")
 					(unit 1)
 				)

Commit message: Chasis minisumo terminado
Parts:
- C45: renamed from C47; footprint Capacitor_SMD:C_0805_2012Metric -> Capacitor_SMD:C_0402_1005Metric
- C46: renamed from C48; footprint Capacitor_SMD:C_0201_0603Metric -> Capacitor_SMD:C_0402_1005Metric
- R33, R34: footprint Resistor_SMD:R_0201_0603Metric -> Resistor_SMD:R_0402_1005Metric
- renumbered J10 to J11, U4 to U5
Connections:
- net +3V0_s: now also U5.3 (A2); no longer U5.4 (A1)
- net GND_s: now also U5.4 (A1); no longer U5.3 (A2)
Changed lines of the file:
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@@
 		)
 	)
-	(label "GND_s"
+	(label "+3V0_s"
 		(at 118.11 92.075 180)
 		(effects
@@
 		)
 	)
-	(label "+3V0_s"
+	(label "GND_s"
 		(at 118.11 89.535 180)
 		(effects
@@
 			)
 		)
-		(property "Footprint" "Resistor_SMD:R_0201_0603Metric"
+		(property "Footprint" "Resistor_SMD:R_0402_1005Metric"
 			(at 111.125 101.473 90)
 			(effects
@@
 		)
 		(property "VACANCIES" ""
+			(at 111.125 99.695 90)
+			(effects
+				(font
+					(size 1.27 1.27)
+				)
+				(hide yes)
+			)
+		)
+		(property "CREATOR" ""
+			(at 111.125 99.695 90)
+			(effects
+				(font
+					(size 1.27 1.27)
+				)
+				(hide yes)
+			)
+		)
+		(property "Sim.Pins" ""
+			(at 111.125 99.695 90)
+			(effects
+				(font
+					(size 1.27 1.27)
+				)
+				(hide yes)
+			)
+		)
+		(property "VERIFIER" ""
 			(at 111.125 99.695 90)
 			(effects
@@
 			)
 		)
-		(property "Footprint" "Resistor_SMD:R_0201_0603Metric"
+		(property "Footprint" "Resistor_SMD:R_0402_1005Metric"
 			(at 111.125 98.933 90)
 			(effects
@@
 		)
 		(property "VACANCIES" ""
+			(at 111.125 97.155 90)
+			(effects
+				(font
+					(size 1.27 1.27)
+				)
+				(hide yes)
+			)
+		)
+		(property "CREATOR" ""
+			(at 111.125 97.155 90)
+			(effects
+				(font
+					(size 1.27 1.27)
+				)
+				(hide yes)
+			)
+		)
+		(property "Sim.Pins" ""
+			(at 111.125 97.155 90)
+			(effects
+				(font
+					(size 1.27 1.27)
+				)
+				(hide yes)
+			)
+		)
+		(property "VERIFIER" ""
 			(at 111.125 97.155 90)
 			(effects
@@
 		(on_board yes)
 		(dnp no)
-		(property "Reference" "C47"
+		(property "Reference" "C45"
 			(at 187.325 88.265 0)
 			(effects
@@
 			)
 		)
-		(property "Footprint" "Capacitor_SMD:C_0805_2012Metric"
+		(property "Footprint" "Capacitor_SMD:C_0402_1005Metric"
 			(at 194.0052 94.615 0)
 			(effects
@@
 		)
 		(property "VACANCIES" ""
+			(at 193.04 90.805 0)
+			(effects
+				(font
+					(size 1.27 1.27)
+				)
+				(hide yes)
+			)
+		)
+		(property "CREATOR" ""
+			(at 193.04 90.805 0)
+			(effects
+				(font
+					(size 1.27 1.27)
+				)
+				(hide yes)
+			)
+		)
+		(property "Sim.Pins" ""
+			(at 193.04 90.805 0)
+			(effects
+				(font
+					(size 1.27 1.27)
+				)
+				(hide yes)
+			)
+		)
+		(property "VERIFIER" ""
 			(at 193.04 90.805 0)
 			(effects
@@
 			(project "Half-Size Micromouse"
 				(path "/96b72c82-8e98-4b00-820e-849de0fa96c7/358c7740-1065-4f93-94de-62d9b382bca9"
-					(reference "C47")
+					(reference "C45")
 					(unit 1)
 				)
@@
 		(dnp no)
 		(fields_autoplaced yes)
-		(property "Reference" "U4"
+		(property "Reference" "U5"
 			(at 143.51 74.295 0)
 			(effects
@@
 		)
 		(property "VACANCIES" ""
+			(at 143.51 97.155 0)
+			(effects
+				(font
+					(size 1.27 1.27)
+				)
+				(hide yes)
+			)
+		)
+		(property "CREATOR" ""
+			(at 143.51 97.155 0)
+			(effects
+				(font
+					(size 1.27 1.27)
+				)
+				(hide yes)
+			)
+		)
+		(property "Sim.Pins" ""
+			(at 143.51 97.155 0)
+			(effects
+				(font
+					(size 1.27 1.27)
+				)
+				(hide yes)
+			)
+		)
+		(property "VERIFIER" ""
 			(at 143.51 97.155 0)
 			(effects
@@
 			(project "Half-Size Micromouse"
 				(path "/96b72c82-8e98-4b00-820e-849de0fa96c7/358c7740-1065-4f93-94de-62d9b382bca9"
-					(reference "U4")
+					(reference "U5")
 					(unit 1)
 				)
@@
 		(on_board yes)
 		(dnp no)
-		(property "Reference" "J10"
+		(property "Reference" "J11"
 			(at 80.645 81.28 0)
 			(effects
@@
 		)
 		(property "VACANCIES" ""
+			(at 79.375 92.075 0)
+			(effects
+				(font
+					(size 1.27 1.27)
+				)
+				(hide yes)
+			)
+		)
+		(property "CREATOR" ""
+			(at 79.375 92.075 0)
+			(effects
+				(font
+					(size 1.27 1.27)
+				)
+				(hide yes)
+			)
+		)
+		(property "Sim.Pins" ""
+			(at 79.375 92.075 0)
+			(effects
+				(font
+					(size 1.27 1.27)
+				)
+				(hide yes)
+			)
+		)
+		(property "VERIFIER" ""
 			(at 79.375 92.075 0)
 			(effects
@@
 			(project "Half-Size Micromouse"
 				(path "/96b72c82-8e98-4b00-820e-849de0fa96c7/358c7740-1065-4f93-94de-62d9b382bca9"
-					(reference "J10")
+					(reference "J11")
 					(unit 1)
 				)
@@
 		(on_board yes)
 		(dnp no)
-		(property "Reference" "C48"
+		(property "Reference" "C46"
 			(at 199.39 88.265 0)
 			(effects
@@
 			)
 		)
-		(property "Footprint" "Capacitor_SMD:C_0201_0603Metric"
+		(property "Footprint" "Capacitor_SMD:C_0402_1005Metric"
 			(at 206.0702 94.615 0)
 			(effects
@@
 		)
 		(property "VACANCIES" ""
+			(at 205.105 90.805 0)
+			(effects
+				(font
+					(size 1.27 1.27)
+				)
+				(hide yes)
+			)
+		)
+		(property "CREATOR" ""
+			(at 205.105 90.805 0)
+			(effects
+				(font
+					(size 1.27 1.27)
+				)
+				(hide yes)
+			)
+		)
+		(property "Sim.Pins" ""
+			(at 205.105 90.805 0)
+			(effects
+				(font
+					(size 1.27 1.27)
+				)
+				(hide yes)
+			)
+		)
+		(property "VERIFIER" ""
 			(at 205.105 90.805 0)
 			(effects
@@
 			(project "Half-Size Micromouse"
 				(path "/96b72c82-8e98-4b00-820e-849de0fa96c7/358c7740-1065-4f93-94de-62d9b382bca9"
-					(reference "C48")
+					(reference "C46")
 					(unit 1)
 				)
