File: Micromouse/MP6551_Der.kicad_sch (KiCad schematic)
At the start: 8 parts, among them IC3 AD8418AWHRZ, M3 MOT_D, U7 MP6551GQB-Z

Commit message: Chasis minisumo terminado
Parts:
- removed C56: 470uF, Capacitor_THT:CP_Radial_D6.3mm_P2.50mm, symbol Device:C_Polarized_US
- removed M3: MOT_D, symbol Motor Coreless:Motor_Coreless_Micromouse
- added C54: APV0609471M010R, CAPAE660X980N, symbol APV0609471M010R:APV0609471M010R
- added J13: MOT_D, JST_SH_2PIN_SMD_VERTICAL:JST_BM02B-SRSS-TB_LF__SN_, symbol BM02B-SRSS-TB_LF__SN_:BM02B-SRSS-TB_LF__SN_
- C52: renamed from C54; value 100nF -> 0.1uF; footprint Capacitor_SMD:C_0201_0603Metric -> Capacitor_SMD:C_0402_1005Metric_Pad0.74x0.62mm_HandSolder
- C53: renamed from C55; footprint Capacitor_SMD:C_0805_2012Metric -> Capacitor_SMD:C_0402_1005Metric_Pad0.74x0.62mm_HandSolder
- R37: footprint Resistor_SMD:R_0201_0603Metric -> Resistor_SMD:R_0402_1005Metric_Pad0.72x0.64mm_HandSolder
- renumbered IC3 to U10, U7 to U9
Connections:
- net SHUNT_MI is gone; now on net SHUNT_MD: R38.1, U9.3 (OUT2_1), U9.8 (OUT2_2)
- net GND: now also C54.2 (-)
- net MOT_D+: now also J13.2
- net POW_IN: now also C54.1 (+)
- net MOT_D-: now reaches U9.1 (OUT1_1), U9.10 (OUT1_2)
- net MOT_D-: now also J13.1
- new net: J13.S1 (SHIELD), J13.S2 (SHIELD)
- no-connect marks 3 -> 4
Other:
- moved on the sheet: C52, C53
