File: Micromouse/MP6551_Izq.kicad_sch (KiCad schematic)
At the start: 8 parts, among them IC2 AD8418AWHRZ, M2 MOT_I, U6 MP6551GQB-Z

Commit message: Chasis minisumo terminado
Parts:
- removed C53: 470uF, Capacitor_THT:CP_Radial_D6.3mm_P2.50mm, symbol Device:C_Polarized_US
- removed M2: MOT_I, symbol Motor Coreless:Motor_Coreless_Micromouse
- added C51: APV0609471M010R, CAPAE660X980N, symbol APV0609471M010R:APV0609471M010R
- added J12: MOT_I, JST_SH_2PIN_SMD_VERTICAL:JST_BM02B-SRSS-TB_LF__SN_, symbol BM02B-SRSS-TB_LF__SN_:BM02B-SRSS-TB_LF__SN_
- C49: renamed from C51; value 100nF -> 0.1uF; footprint Capacitor_SMD:C_0201_0603Metric -> Capacitor_SMD:C_0402_1005Metric_Pad0.74x0.62mm_HandSolder
- C50: renamed from C52; footprint Capacitor_SMD:C_0805_2012Metric -> Capacitor_SMD:C_0402_1005Metric_Pad0.74x0.62mm_HandSolder
- R35: footprint Resistor_SMD:R_0201_0603Metric -> Resistor_SMD:R_0402_1005Metric_Pad0.72x0.64mm_HandSolder
- renumbered U6 to U7, IC2 to U8
Connections:
- net GND: now also C51.2 (-)
- net MOT_I-: now also J12.1
- net POW_IN: now also C51.1 (+)
- net MOT_I+: now reaches U7.3 (OUT2_1), U7.8 (OUT2_2)
- net MOT_I+: now also J12.2
- new net: J12.S1 (SHIELD), J12.S2 (SHIELD)
- no-connect marks 3 -> 4
