File: Micromouse/LSM6DSRTR.kicad_sch (KiCad schematic)
At the start: 3 parts, among them U5 LSM6DSRTR

Commit message: Chasis minisumo terminado
Parts:
- C47: renamed from C49; value 100nF -> 0.1uF; footprint Capacitor_SMD:C_0201_0603Metric -> Capacitor_SMD:C_0402_1005Metric_Pad0.74x0.62mm_HandSolder
- C48: renamed from C50; value 100nF -> 0.1uF; footprint Capacitor_SMD:C_0201_0603Metric -> Capacitor_SMD:C_0402_1005Metric_Pad0.74x0.62mm_HandSolder
- renumbered U5 to U6
Changed lines of the file:
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@@
 		(on_board yes)
 		(dnp no)
-		(property "Reference" "#PWR061"
+		(property "Reference" "#PWR060"
 			(at 193.04 98.425 0)
 			(effects
@@
 			(project "Micromouse"
 				(path "/96b72c82-8e98-4b00-820e-849de0fa96c7/48901c7f-a0cf-4078-a2bc-b3b72fecfd57"
-					(reference "#PWR061")
+					(reference "#PWR060")
 					(unit 1)
 				)
@@
 		(dnp no)
 		(fields_autoplaced yes)
-		(property "Reference" "#PWR062"
+		(property "Reference" "#PWR061"
 			(at 193.04 114.3 0)
 			(effects
@@
 			(project "Micromouse"
 				(path "/96b72c82-8e98-4b00-820e-849de0fa96c7/48901c7f-a0cf-4078-a2bc-b3b72fecfd57"
-					(reference "#PWR062")
+					(reference "#PWR061")
 					(unit 1)
 				)
@@
 		(dnp no)
 		(fields_autoplaced yes)
-		(property "Reference" "U5"
+		(property "Reference" "U6"
 			(at 153.67 71.12 0)
 			(effects
@@
 		)
 		(property "VACANCIES" ""
+			(at 128.27 81.28 0)
+			(effects
+				(font
+					(size 1.27 1.27)
+				)
+				(hide yes)
+			)
+		)
+		(property "CREATOR" ""
+			(at 128.27 81.28 0)
+			(effects
+				(font
+					(size 1.27 1.27)
+				)
+				(hide yes)
+			)
+		)
+		(property "Sim.Pins" ""
+			(at 128.27 81.28 0)
+			(effects
+				(font
+					(size 1.27 1.27)
+				)
+				(hide yes)
+			)
+		)
+		(property "VERIFIER" ""
 			(at 128.27 81.28 0)
 			(effects
@@
 			(project "Micromouse"
 				(path "/96b72c82-8e98-4b00-820e-849de0fa96c7/48901c7f-a0cf-4078-a2bc-b3b72fecfd57"
-					(reference "U5")
+					(reference "U6")
 					(unit 1)
 				)
@@
 		(on_board yes)
 		(dnp no)
-		(property "Reference" "C49"
+		(property "Reference" "C47"
 			(at 115.8875 103.1875 0)
 			(effects
@@
 			)
 		)
-		(property "Value" "100nF"
+		(property "Value" "0.1uF"
 			(at 117.1575 100.6475 0)
 			(effects
@@
 			)
 		)
-		(property "Footprint" "Capacitor_SMD:C_0201_0603Metric"
+		(property "Footprint" "Capacitor_SMD:C_0402_1005Metric_Pad0.74x0.62mm_HandSolder"
 			(at 108.2548 99.695 0)
 			(effects
@@
 		)
 		(property "VACANCIES" ""
+			(at 109.22 103.505 0)
+			(effects
+				(font
+					(size 1.27 1.27)
+				)
+				(hide yes)
+			)
+		)
+		(property "CREATOR" ""
+			(at 109.22 103.505 0)
+			(effects
+				(font
+					(size 1.27 1.27)
+				)
+				(hide yes)
+			)
+		)
+		(property "Sim.Pins" ""
+			(at 109.22 103.505 0)
+			(effects
+				(font
+					(size 1.27 1.27)
+				)
+				(hide yes)
+			)
+		)
+		(property "VERIFIER" ""
 			(at 109.22 103.505 0)
 			(effects
@@
 			(project "Micromouse"
 				(path "/96b72c82-8e98-4b00-820e-849de0fa96c7/48901c7f-a0cf-4078-a2bc-b3b72fecfd57"
-					(reference "C49")
+					(reference "C47")
 					(unit 1)
 				)
@@
 		(on_board yes)
 		(dnp no)
-		(property "Reference" "#PWR060"
+		(property "Reference" "#PWR059"
 			(at 109.22 85.09 0)
 			(effects
@@
 			(project "Micromouse"
 				(path "/96b72c82-8e98-4b00-820e-849de0fa96c7/48901c7f-a0cf-4078-a2bc-b3b72fecfd57"
-					(reference "#PWR060")
+					(reference "#PWR059")
 					(unit 1)
 				)
@@
 		(dnp no)
 		(fields_autoplaced yes)
-		(property "Reference" "#PWR059"
+		(property "Reference" "#PWR058"
 			(at 104.14 116.205 0)
 			(effects
@@
 			(project "Micromouse"
 				(path "/96b72c82-8e98-4b00-820e-849de0fa96c7/48901c7f-a0cf-4078-a2bc-b3b72fecfd57"
-					(reference "#PWR059")
+					(reference "#PWR058")
 					(unit 1)
 				)
@@
 		(on_board yes)
 		(dnp no)
-		(property "Reference" "C50"
+		(property "Reference" "C48"
 			(at 199.7075 101.9175 0)
 			(effects
@@
 			)
 		)
-		(property "Value" "100nF"
+		(property "Value" "0.1uF"
 			(at 200.9775 99.3775 0)
 			(effects
@@
 			)
 		)
-		(property "Footprint" "Capacitor_SMD:C_0201_0603Metric"
+		(property "Footprint" "Capacitor_SMD:C_0402_1005Metric_Pad0.74x0.62mm_HandSolder"
 			(at 192.0748 98.425 0)
 			(effects
@@
 		)
 		(property "VACANCIES" ""
+			(at 193.04 102.235 0)
+			(effects
+				(font
+					(size 1.27 1.27)
+				)
+				(hide yes)
+			)
+		)
+		(property "CREATOR" ""
+			(at 193.04 102.235 0)
+			(effects
+				(font
+					(size 1.27 1.27)
+				)
+				(hide yes)
+			)
+		)
+		(property "Sim.Pins" ""
+			(at 193.04 102.235 0)
+			(effects
+				(font
+					(size 1.27 1.27)
+				)
+				(hide yes)
+			)
+		)
+		(property "VERIFIER" ""
 			(at 193.04 102.235 0)
 			(effects
@@
 			(project "Micromouse"
 				(path "/96b72c82-8e98-4b00-820e-849de0fa96c7/48901c7f-a0cf-4078-a2bc-b3b72fecfd57"
-					(reference "C50")
+					(reference "C48")
 					(unit 1)
 				)

Commit message: Red 3V0 cambiada a 3V3
Connections:
- net +3V0 renamed +3V3
Changed lines of the file:
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@@
 			)
 		)
-		(property "Value" "+3V0"
+		(property "Value" "+3V3"
 			(at 193.04 89.535 0)
 			(effects
@@
 			)
 		)
-		(property "Value" "+3V0"
+		(property "Value" "+3V3"
 			(at 109.22 76.2 0)
 			(effects
