File: Micromouse/Micromouse.kicad_pcb (KiCad board)
At the start: 2 copper layers, 88.3 x 94 mm, 73 parts, among them IC1 MP6551GQB-Z, J1 ST-LINK, J8 Lipo, J9 AS5048_Izq, Q4 SFH_309-4_5, Q5 SFH_309-4_5, Q8 SFH_309-4_5, Q9 SFH_309-4_5, U1 STM32F405RGTx, U2 CUS-12TB, U3 MP2359DJ-LF-Z, U4 AS5048B-HTSP, U6 LSM6DSRTR, Y1 32.768kHz, Y2 25MHz

Commit message: Commit4
Parts:
- removed J1: ST-LINK, S4B-XH-SM4-TB:JST_S4B-XH-SM4-TB
- removed Y2: 25MHz, Crystal25MHz:XTAL_C3E-25.000-12-3030-X-R
- added C25: 20pF, Capacitor_SMD:C_0201_0603Metric, F.Cu at (211.1, 102.0)
- added C26: 0.1uF, Capacitor_SMD:C_0201_0603Metric, F.Cu at (211.1, 103.7)
- added C32: 10uF, Capacitor_SMD:C_0201_0603Metric, F.Cu at (211.1, 110.7)
- added C33: 1uF, Capacitor_SMD:C_0201_0603Metric, F.Cu at (211.1, 112.5)
- added C34: 0.1uF, Capacitor_SMD:C_0402_1005Metric_Pad0.74x0.62mm_HandSolder, F.Cu at (205.7, 116.0)
- added C35: 10uF, Capacitor_SMD:C_1206_3216Metric, F.Cu at (214.7, 115.0)
- added C36: 10uF, Capacitor_SMD:C_1206_3216Metric, F.Cu at (214.7, 118.4)
- added C37: 0.1uF, Capacitor_SMD:C_0402_1005Metric_Pad0.74x0.62mm_HandSolder, F.Cu at (205.7, 118.0)
- added C38: 1uF, Capacitor_SMD:C_0402_1005Metric_Pad0.74x0.62mm_HandSolder, F.Cu at (205.7, 119.9)
- added C39: 0.1uF, Capacitor_SMD:C_0201_0603Metric, F.Cu at (213.6, 102.0)
- added C40: 10nF, Capacitor_SMD:C_0201_0603Metric, F.Cu at (213.6, 103.7)
- added C41: 10uF, Capacitor_SMD:C_0402_1005Metric_Pad0.74x0.62mm_HandSolder, F.Cu at (205.7, 121.9)
- added C42: 22uF, Capacitor_SMD:C_1206_3216Metric, F.Cu at (214.7, 121.7)
- added C43: 22uF, Capacitor_SMD:C_1206_3216Metric, F.Cu at (214.7, 125.1)
- added C44: 0.1uF, Capacitor_SMD:C_0201_0603Metric, F.Cu at (213.6, 105.5)
- added C45: 10uF, Capacitor_SMD:C_0805_2012Metric, F.Cu at (227.2, 94.8)
- added C46: 0.1uF, Capacitor_SMD:C_0201_0603Metric, F.Cu at (235.5, 87.5)
- added C47: 10uF, Capacitor_SMD:C_0805_2012Metric, F.Cu at (227.2, 106.5)
- added C48: 0.1uF, Capacitor_SMD:C_0201_0603Metric, F.Cu at (235.5, 99.2)
- added C49: 100nF, Capacitor_SMD:C_0201_0603Metric, F.Cu at (231.3, 110.8)
- added C50: 100nF, Capacitor_SMD:C_0201_0603Metric, F.Cu at (231.3, 112.6)
- added C51: 100nF, Capacitor_SMD:C_0201_0603Metric, F.Cu at (232.3, 131.7)
- added C52: 10uF, Capacitor_SMD:C_0805_2012Metric, F.Cu at (220.0, 143.8)
- added C53: 470uF, Capacitor_THT:CP_Radial_D6.3mm_P2.50mm, F.Cu at (229.0, 139.6)
- added C54: 100nF, Capacitor_SMD:C_0201_0603Metric, F.Cu at (213.8, 131.7)
- added C55: 10uF, Capacitor_SMD:C_0805_2012Metric, F.Cu at (201.5, 143.8)
- added C56: 470uF, Capacitor_THT:CP_Radial_D6.3mm_P2.50mm, F.Cu at (210.6, 139.6)
- added C57: 10uF, Capacitor_SMD:C_1206_3216Metric, F.Cu at (187.1, 132.5)
- added C58: 10uF, Capacitor_SMD:C_1206_3216Metric, F.Cu at (187.1, 135.8)
- added C59: 0.1uF, Capacitor_SMD:C_0201_0603Metric, F.Cu at (191.1, 143.5)
- added C60: 0.1uF, Capacitor_SMD:C_0201_0603Metric, F.Cu at (191.1, 145.2)
- added C61: 10uF, Capacitor_SMD:C_1206_3216Metric, F.Cu at (187.1, 139.2)
- added C62: 10uF, Capacitor_SMD:C_1206_3216Metric, F.Cu at (187.1, 142.5)
- added C63: 0.1uF, Capacitor_SMD:C_0201_0603Metric, F.Cu at (191.1, 147.0)
- added C64: 0.1uF, Capacitor_SMD:C_0201_0603Metric, F.Cu at (191.1, 148.7)
- added D1: 1N4148WS, 1N4148WS:SODFL2512X100N, F.Cu at (220.1, 111.6)
- added D12: LTST-G563ZEGBW, RGB5050:LED_LTST-G563ZEGBW, F.Cu at (183.6, 119.9)
- added D13: LED, LED_SMD:LED_0805_2012Metric, F.Cu at (195.5, 102.6)
- added D14: LED, LED_SMD:LED_0805_2012Metric, F.Cu at (195.5, 105.6)
- added D15: LED, LED_SMD:LED_0805_2012Metric, F.Cu at (195.5, 108.7)
- added D16: LED, LED_SMD:LED_0805_2012Metric, F.Cu at (195.5, 111.7)
- added D17: LED, LED_SMD:LED_0805_2012Metric, F.Cu at (195.5, 114.8)
- added D2: 1N5819HW-7, 1N5819HW-7:SOD3715X145N, F.Cu at (183.0, 108.5)
- added D3: LED, LED_SMD:LED_0402_1005Metric_Pad0.77x0.64mm_HandSolder, F.Cu at (210.8, 96.6)
- added D4: LED, LED_SMD:LED_0402_1005Metric_Pad0.77x0.64mm_HandSolder, F.Cu at (210.8, 98.6)
- added D5: LED, LED_SMD:LED_0805_2012Metric, F.Cu at (191.0, 102.6)
- added D6: LED, LED_SMD:LED_0805_2012Metric, F.Cu at (191.0, 105.6)
- added IC2: AD8418AWHRZ, AD8418AWHRZ:SOIC127P600X175-8N, F.Cu at (222.0, 139.0)
- added IC3: AD8418AWHRZ, AD8418AWHRZ:SOIC127P600X175-8N, F.Cu at (203.5, 139.0)
- added J10: AS5048_Der, MicromouseHuellas:Encoder1, F.Cu at (232.6, 106.0)
- added J5: ST_LINK, JST_SH_6PIN_SMD_HORIZONTAL:JST_SM06B-SRSS-TB_LF__SN_, F.Cu at (217.8, 88.2)
- added JP1: SolderJumper_2_Open, Jumper:SolderJumper-2_P1.3mm_Open_RoundedPad1.0x1.5mm, F.Cu at (220.6, 95.5)
- added LS1: Buzzer, CMT-0502-03-SMT-TR:CMT050203SMTTR, F.Cu at (229.7, 118.5)
- added Q1: AO3400A, Package_TO_SOT_SMD:SOT-23, F.Cu at (220.0, 115.6)
- added Q12: AON7423, AON7423:AON7423, F.Cu at (230.8, 125.6)
- added Q2: AO3400A, Package_TO_SOT_SMD:SOT-23, F.Cu at (220.0, 120.0)
- added Q3: AON7423, Package_DFN_QFN:DFN-8-1EP_3x3mm_P0.65mm_EP1.55x2.4mm, F.Cu at (110.1, 83.8)
- added Q4: AO3400A, Package_TO_SOT_SMD:SOT-23, F.Cu at (181.8, 133.0)
- added Q5: AO3400A, Package_TO_SOT_SMD:SOT-23, F.Cu at (181.8, 137.5)
- added Q8: AO3400A, Package_TO_SOT_SMD:SOT-23, F.Cu at (181.8, 141.9)
- added Q9: AO3400A, Package_TO_SOT_SMD:SOT-23, F.Cu at (181.8, 146.4)
- added R1: 10k, Resistor_SMD:R_0201_0603Metric, F.Cu at (213.6, 107.2)
- added R10: 330, Resistor_SMD:R_0402_1005Metric_Pad0.72x0.64mm_HandSolder, F.Cu at (199.3, 112.0)
- added R19: 82, Resistor_SMD:R_0201_0603Metric, F.Cu at (216.0, 103.7)
- added R2: 47K, Resistor_SMD:R_0402_1005Metric_Pad0.72x0.64mm_HandSolder, F.Cu at (199.3, 102.1)
- added R20: 10, Resistor_SMD:R_0201_0603Metric, F.Cu at (216.0, 105.5)
- added R27: 330, Resistor_SMD:R_0402_1005Metric_Pad0.72x0.64mm_HandSolder, F.Cu at (205.8, 108.0)
- added R28: 100K, Resistor_SMD:R_0402_1005Metric_Pad0.72x0.64mm_HandSolder, F.Cu at (205.8, 110.0)
- added R29: 33K, Resistor_SMD:R_0402_1005Metric_Pad0.72x0.64mm_HandSolder, F.Cu at (205.8, 112.0)
- added R30: 4.7K, Resistor_SMD:R_0402_1005Metric_Pad0.72x0.64mm_HandSolder, F.Cu at (205.8, 114.0)
- added R31: 4.7k, Resistor_SMD:R_0201_0603Metric, F.Cu at (235.5, 89.3)
- added R32: 4.7k, Resistor_SMD:R_0201_0603Metric, F.Cu at (235.5, 91.0)
- added R33: 4.7k, Resistor_SMD:R_0201_0603Metric, F.Cu at (235.5, 100.9)
- added R34: 4.7k, Resistor_SMD:R_0201_0603Metric, F.Cu at (235.5, 102.7)
- added R35: 10k, Resistor_SMD:R_0201_0603Metric, F.Cu at (232.3, 133.4)
- added R36: 0.05, Resistor_SMD:R_2512_6332Metric, F.Cu at (222.1, 133.3)
- added R37: 10k, Resistor_SMD:R_0201_0603Metric, F.Cu at (213.8, 133.4)
- added R38: 0.05, Resistor_SMD:R_2512_6332Metric, F.Cu at (203.6, 133.3)
- added R39: 4.7k, Resistor_SMD:R_0201_0603Metric, F.Cu at (193.6, 143.5)
- added R4: 220, Resistor_SMD:R_0201_0603Metric, F.Cu at (213.6, 109.0)
- added R40: 4.7k, Resistor_SMD:R_0201_0603Metric, F.Cu at (193.6, 145.2)
- added R41: 30, Resistor_SMD:R_0805_2012Metric, F.Cu at (192.1, 132.3)
- added R42: 30, Resistor_SMD:R_0805_2012Metric, F.Cu at (192.1, 135.2)
- added R43: 1.5k, Resistor_SMD:R_0201_0603Metric, F.Cu at (193.6, 147.0)
- added R44: 1.5k, Resistor_SMD:R_0201_0603Metric, F.Cu at (193.6, 148.7)
- added R45: 4.7k, Resistor_SMD:R_0201_0603Metric, F.Cu at (196.0, 143.5)
- added R46: 4.7k, Resistor_SMD:R_0201_0603Metric, F.Cu at (196.0, 145.2)
- added R47: 30, Resistor_SMD:R_0805_2012Metric, F.Cu at (192.1, 138.2)
- added R48: 30, Resistor_SMD:R_0805_2012Metric, F.Cu at (192.1, 141.1)
- added R49: 1.5k, Resistor_SMD:R_0201_0603Metric, F.Cu at (196.0, 147.0)
- added R5: 10k, Resistor_SMD:R_0201_0603Metric, F.Cu at (213.6, 110.7)
- added R50: 1.5k, Resistor_SMD:R_0201_0603Metric, F.Cu at (196.0, 148.7)
- added R6: 10k, Resistor_SMD:R_0201_0603Metric, F.Cu at (213.6, 112.5)
- added R7: 1K, Resistor_SMD:R_0402_1005Metric_Pad0.72x0.64mm_HandSolder, F.Cu at (199.3, 106.1)
- added R8: 10K, Resistor_SMD:R_0402_1005Metric_Pad0.72x0.64mm_HandSolder, F.Cu at (199.3, 108.0)
- added R9: 47k, Resistor_SMD:R_0402_1005Metric_Pad0.72x0.64mm_HandSolder, F.Cu at (199.3, 110.0)
- added S4: BTN_2, PTS636_SM43J_SMTR_LFS:SW_PTS636_SM43J_SMTR_LFS, F.Cu at (184.3, 99.3)
- added S5: BTN_3, PTS636_SM43J_SMTR_LFS:SW_PTS636_SM43J_SMTR_LFS, F.Cu at (184.3, 104.3)
- added U5: LSM6DSRTR, LSM6DSRTR:PQFN50P250X300X86-14N, F.Cu at (227.8, 112.0)
- added U7: MP6551GQB-Z, MP6551GQB-Z:MP6551GQBZ, F.Cu at (210.5, 133.1)
- C1, C3: value 12.5pF -> 2.2uF; footprint Capacitor_SMD:C_0201_0603Metric -> Capacitor_SMD:C_0805_2012Metric
- C10, C6: value 0.1uF -> 1uF; footprint Capacitor_SMD:C_0201_0603Metric -> Capacitor_SMD:C_0402_1005Metric_Pad0.74x0.62mm_HandSolder
- C12: value 0.1uF -> 0.1uf; footprint Capacitor_SMD:C_0201_0603Metric -> Capacitor_SMD:C_0402_1005Metric_Pad0.74x0.62mm_HandSolder
- C13: value 0.1uF -> 47uF; footprint Capacitor_SMD:C_0201_0603Metric -> Capacitor_SMD:C_0805_2012Metric
- C14: value 0.1uF -> 20pF
- C15: value 10nF -> 47uF; footprint Capacitor_SMD:C_0201_0603Metric -> Capacitor_SMD:C_0805_2012Metric
- C16: value 20pF -> 1uF
- C17: value 0.1uF -> 10uF; footprint Capacitor_SMD:C_0201_0603Metric -> Capacitor_SMD:C_0402_1005Metric_Pad0.74x0.62mm_HandSolder
- C18: value 22uF -> 0.1uF; footprint Capacitor_SMD:C_1206_3216Metric -> Capacitor_SMD:C_0201_0603Metric
- C19: footprint Capacitor_SMD:C_1206_3216Metric -> Capacitor_SMD:C_0201_0603Metric
- C2, C4: value 2.2uF -> 0.1uF; footprint Capacitor_SMD:C_0805_2012Metric -> Capacitor_SMD:C_0402_1005Metric_Pad0.74x0.62mm_HandSolder
- C20: value 22uF -> 10uF; footprint Capacitor_SMD:C_1206_3216Metric -> Capacitor_SMD:C_0402_1005Metric_Pad0.74x0.62mm_HandSolder
- C21: value 20pF -> 10uF; footprint Capacitor_SMD:C_0201_0603Metric -> Capacitor_SMD:C_0402_1005Metric_Pad0.74x0.62mm_HandSolder
- C23: footprint Capacitor_SMD:C_0805_2012Metric -> Capacitor_SMD:C_0201_0603Metric; moved to F.Cu
- C24: value 0.1uF -> 10uF; footprint Capacitor_SMD:C_0201_0603Metric -> Capacitor_SMD:C_0402_1005Metric_Pad0.74x0.62mm_HandSolder; moved to F.Cu
- C27: value 100nF -> 10uF
- C28: value 100nF -> 0.01uF
- C29: value 100nF -> 10uF; footprint Capacitor_SMD:C_0201_0603Metric -> Capacitor_SMD:C_0402_1005Metric_Pad0.74x0.62mm_HandSolder
- C30: value 10uF -> 47uF
- C31: value 470uF -> 0.1uF; footprint Capacitor_THT:CP_Radial_D6.3mm_P2.50mm -> Capacitor_SMD:C_0201_0603Metric
- C5: value 1uF -> 0.1uF; footprint Capacitor_SMD:C_0201_0603Metric -> Capacitor_SMD:C_0402_1005Metric_Pad0.74x0.62mm_HandSolder
- C7: value 0.01uF -> 0.1uF; footprint Capacitor_SMD:C_0201_0603Metric -> Capacitor_SMD:C_0402_1005Metric_Pad0.74x0.62mm_HandSolder
- C8: value 1uF -> 4.7uF; footprint Capacitor_SMD:C_0201_0603Metric -> Capacitor_SMD:C_0402_1005Metric_Pad0.74x0.62mm_HandSolder
- C9: footprint Capacitor_SMD:C_0201_0603Metric -> Capacitor_SMD:C_0402_1005Metric_Pad0.74x0.62mm_HandSolder
- D11: value LED -> 1N5819HW-7; footprint LED_SMD:LED_0201_0603Metric -> 1N5819HW-7:SOD3715X145N
- D7, D8: footprint LED_SMD:LED_0805_2012Metric_Pad1.15x1.40mm_HandSolder -> LED_SMD:LED_0805_2012Metric
- D9: value 1N5819HW-7 -> LED; footprint 1N5819HW-7:SOD3715X145N -> LED_SMD:LED_0805_2012Metric
- IC1: value MP6551GQB-Z -> ME6211C30M5G; footprint KiCad:MP6551GQBZ -> ME6211C33M5G:SOT95P282X145-5N
- Q10: renamed from Q8; value SFH_309-4_5 -> SFH_309FA
- Q11: renamed from Q9; value SFH_309-4_5 -> SFH_309FA
- Q6: renamed from Q4; value SFH_309-4_5 -> SFH_309FA
- Q7: renamed from Q5; value SFH_309-4_5 -> SFH_309FA
- R11, R12: value 220 -> 330; footprint Resistor_SMD:R_0201_0603Metric -> Resistor_SMD:R_0402_1005Metric_Pad0.72x0.64mm_HandSolder
- R13: value 10k -> 330; footprint Resistor_SMD:R_0805_2012Metric -> Resistor_SMD:R_0402_1005Metric_Pad0.72x0.64mm_HandSolder
- R14: value 4.7k -> 330; footprint Resistor_SMD:R_0201_0603Metric -> Resistor_SMD:R_0402_1005Metric_Pad0.72x0.64mm_HandSolder
- R15, R23: value 10k -> 330; footprint Resistor_SMD:R_0201_0603Metric -> Resistor_SMD:R_0402_1005Metric_Pad0.72x0.64mm_HandSolder
- R16: value 27k -> 1K; footprint Resistor_SMD:R_0201_0603Metric -> Resistor_SMD:R_0402_1005Metric_Pad0.72x0.64mm_HandSolder
- R17: value 4.7k -> 47K; footprint Resistor_SMD:R_0201_0603Metric -> Resistor_SMD:R_0402_1005Metric_Pad0.72x0.64mm_HandSolder; moved to F.Cu
- R18: value 4.7k -> 10k; moved to F.Cu
- R21: value 10k -> 22
- R22: value 10k -> 51k
- R24, R25: value 4.99k -> 330; footprint Resistor_SMD:R_0201_0603Metric -> Resistor_SMD:R_0402_1005Metric_Pad0.72x0.64mm_HandSolder
- R26: value 499 -> 330; footprint Resistor_SMD:R_0201_0603Metric -> Resistor_SMD:R_0402_1005Metric_Pad0.72x0.64mm_HandSolder
- R3: value 10k -> 27K; footprint Resistor_SMD:R_0201_0603Metric -> Resistor_SMD:R_0402_1005Metric_Pad0.72x0.64mm_HandSolder
- S1: value ButtonS -> CUS-12TB; footprint PTS636_SM43J_SMTR_LFS:SW_PTS636_SM43J_SMTR_LFS -> CUS-12TB:CUS-12B
- S3: value ButtonC -> BTN_1
- U2: value CUS-12TB -> MP2359DJ-LF-Z; footprint CUS-12TB:CUS-12B -> MP2359DJ-LF-Z:SOT95P280X100-6N
- U3: value MP2359DJ-LF-Z -> AS5048B-HTSP; footprint MP2359DJ-LF-Z:SOT95P280X100-6N -> AS5048B-HTSP:SOP65P640X120-14N
- U6: value LSM6DSRTR -> MP6551GQB-Z; footprint footprints:LGA-14L_2P5X3X0P83_STM-M -> MP6551GQB-Z:MP6551GQBZ
- Y1: value 32.768kHz -> 8MHz; footprint CC5V-T1A_32.768KHZ_12.5PF_20PPM_TA_QC:XTAL_CC5V-T1A_32.768KHZ_12.5PF_20PPM_TA_QC -> 8.000MHz3.2x2.5mm:XTAL_C3E-8.000-18-3030-R
- moved J9 188.1 mm to (232.6, 94.4)
- moved U4 185.6 mm to (229.9, 101.6), turned to 0 degrees
- moved R18 173.3 mm to (216.0, 102.0), turned to 0 degrees
- moved C24 168.8 mm to (202.5, 125.8)
- moved C23 166.9 mm to (208.7, 112.5)
- moved Y1 159.7 mm to (220.3, 103.3), turned to 0 degrees
- moved R17 157.3 mm to (202.6, 112.0), turned to 0 degrees
- moved FB1 147.9 mm to (219.1, 123.4)
- moved C3 145.2 mm to (209.7, 117.8), turned to 0 degrees
- moved C1 145.2 mm to (209.7, 114.8), turned to 0 degrees
- moved C16 144.2 mm to (208.7, 105.5), turned to 0 degrees
- moved U6 139.1 mm to (229.0, 133.1)
- moved C21 139.1 mm to (202.5, 123.9), turned to 0 degrees
- moved C2 136.4 mm to (199.3, 116.0), turned to 0 degrees
- moved C31 133.7 mm to (211.1, 109.0), turned to 0 degrees
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- renumbered D12 to D18, D13 to D19, D14 to D20, D15 to D21
Connections:
- net SCL_1 renamed SCL_s
- net SDA_1 renamed SDA_s
- C1 pad 1: Net-(U1-PC14) -> Net-(U1-VCAP_1)
- C1 pad 2: GND -> VSS
- C10 pad 1: RUN -> VSS
- C10 pad 2: GND -> VBAT
- C11 pad 1: +3V0 -> VBAT
- C11 pad 2: GND -> VSS
- C12 pad 1: +3V0 -> +5V
- C12 pad 2: GND -> VSS
- C13 pad 1: +3V0 -> VSS
- C13 pad 2: GND -> POW_IN
- C14 pad 1: +3V0 -> RCC_OSC_IN
- C14 pad 2: GND -> VSS
- C15 pad 1: Net-(U3-BST) -> VSS
- C15 pad 2: Net-(U3-SW) -> POW_IN
- C16 pad 1: RCC_OSC_IN -> VBAT
- C16 pad 2: GND -> VSS
- C17 pad 1: +3V0 -> VSS
- C17 pad 2: GND -> VBAT
- C18 pad 1: Net-(C18-Pad1) -> VBAT
- C18 pad 2: +3V0(BAT) -> VSS
- C19 pad 1: +3V0 -> +5V
- C19 pad 2: GND -> VSS
- C2 pad 1: Net-(U1-VCAP_1) -> VSS
- C2 pad 2: GND -> VBAT
- C20 pad 1: +3V0(BAT) -> VSS
- C20 pad 2: GND -> POW_IN
- C21 pad 1: RCC_OSC_OUT -> VSS
- C21 pad 2: GND -> POW_IN
- C22 pad 1: +3V0(BAT) -> VBAT
- C22 pad 2: GND -> VSS
- C23 pad 1: /AS5048_Izq/+3V0_s -> +5V
- C23 pad 2: /AS5048_Izq/GND_s -> VSS
- C24 pad 1: /AS5048_Izq/+3V0_s -> VSS
- C24 pad 2: /AS5048_Izq/GND_s -> POW_IN
- C27 pad 1: GND -> +5V
- C27 pad 2: +3V0 -> VSS
- C28 pad 1: GND -> VBAT
- C28 pad 2: +3V0 -> VSS
- C29 pad 1: GND -> VSS
- C3 pad 1: Net-(U1-PC15) -> Net-(U1-VCAP_2)
- C3 pad 2: GND -> VSS
- C30 pad 1: GND -> VSS
- C31 pad 1: POW_IN -> VBAT
- C31 pad 2: GND -> VSS
- C4 pad 1: Net-(U1-VCAP_2) -> VSS
- C4 pad 2: GND -> VBAT
- C5 pad 1: +3V0 -> VSS
- C5 pad 2: GND -> VBAT
- C6 pad 1: SEL -> VSS
- C6 pad 2: GND -> VBAT
- C7 pad 1: 3V0A -> VSS
- C7 pad 2: GND -> VBAT
- C8 pad 1: 3V0A -> VSS
- C8 pad 2: GND -> VBAT
- C9 pad 1: NRST -> VSS
- C9 pad 2: GND -> VBAT
- D10 pad A: GND -> VSS
- D10 pad C: Net-(U3-SW) -> Net-(U2-SW)
- D7 pad 1: Net-(D7-K) -> VSS
- D7 pad 2: +3V0 -> Net-(D7-A)
- D8 pad 1: Net-(D8-K) -> VSS
- D8 pad 2: SEL_LED -> Net-(D8-A)
- FB1 pad 1: +3V0 -> VBAT
- FB1 pad 2: 3V0A -> VBAT
- IC1 pad 1: Net-(IC1-OUT1_1) -> +5V
- IC1 pad 2: POW_IN -> VSS
- IC1 pad 3: Net-(IC1-OUT2_1) -> +5V
- IC1 pad 4: /MP6551/EN2 -> unconnected-(IC1-NC-Pad4)
- IC1 pad 5: /MP6551/IN2 -> VBAT
- J8 pad 1: POW_IN -> LIPO
- J8 pad 2: GND -> VSS
- L1 pad 1: Net-(U3-SW) -> Net-(U2-SW)
- L1 pad 2: Net-(C18-Pad1) -> Net-(C42-Pad1)
- R11 pad 1: Net-(D7-K) -> LED_1
- R11 pad 2: GND -> Net-(D5-A)
- R12 pad 1: GND -> LED_2
- R12 pad 2: Net-(D8-K) -> Net-(D6-A)
- R13 pad 1: POW_IN -> LED_3
- R13 pad 2: BAT_VOL -> Net-(D7-A)
- R14 pad 1: BAT_VOL -> LED_4
- R14 pad 2: GND -> Net-(D8-A)
- R15 pad 1: Net-(U3-FB) -> LED_5
- R15 pad 2: GND -> Net-(D9-A)
- R16 pad 1: Net-(U3-FB) -> +3V3
- R16 pad 2: Net-(C18-Pad1) -> Net-(D4-A)
- R17 pad 1: /AS5048_Izq/+3V0_s -> VSS
- R17 pad 2: /AS5048_Izq/SCL_s -> MENU_ESTADO
- R18 pad 1: /AS5048_Izq/+3V0_s -> Net-(U2-FB)
- R18 pad 2: /AS5048_Izq/SDA_s -> VSS
- R21 pad 1: SDA -> LED_B
- R21 pad 2: +3V0 -> Net-(D12-Pad6)
- R22 pad 1: SCL -> Net-(U2-FB)
- R22 pad 2: +3V0 -> Net-(C42-Pad1)
- R23 pad 1: GND -> LED_6
- R23 pad 2: Net-(IC1-SR) -> Net-(D13-A)
- R24 pad 1: /MP6551/CM1 -> LED_7
- R24 pad 2: GND -> Net-(D14-A)
- R25 pad 1: /MP6551/CM2 -> LED_8
- R25 pad 2: GND -> Net-(D15-A)
- R26 pad 1: +3V0 -> LED_9
- R26 pad 2: Net-(D11-A) -> Net-(D16-A)
- R3 pad 1: GND -> BAT_VOLTAGE
- R3 pad 2: Net-(U1-BOOT0) -> VSS
- S2 pad 2: GND -> VSS
- S3 pad 1: RUN -> MENU_ESTADO
- S3 pad 2: GND -> Net-(R28-Pad2)
- U1 pad 1: +3V0 -> VBAT
- U1 pad 10: SEL_LED -> IR_REC_2
- U1 pad 11: EN2 -> IR_REC_3
- U1 pad 12: GND -> VSS
- U1 pad 13: 3V0A -> VBAT
- U1 pad 14: BAT_VOL -> IR_POW_4
- U1 pad 15: IR_REC_1 -> IR_POW_1
- U1 pad 16: PWM_FAN -> IR_POW_2
- U1 pad 17: EN1 -> IR_POW_3
- U1 pad 18: GND -> VSS
- U1 pad 19: +3V0 -> VBAT
- U1 pad 2: unconnected-(U1-PC13-Pad2) -> LED_8
- U1 pad 20: IR_REC_2 -> BAT_VOLTAGE
- U1 pad 21: IR_REC_3 -> CURRENT_MD
- U1 pad 22: CM1 -> CURRENT_MI
- U1 pad 23: IR_REC_4 -> MENU_ESTADO
- U1 pad 24: CM2 -> LED_1
- U1 pad 25: IN2 -> LED_2
- U1 pad 26: unconnected-(U1-PB0-Pad26) -> LED_3
- U1 pad 27: unconnected-(U1-PB1-Pad27) -> LED_4
- U1 pad 28: NFAULT -> LED_5
- U1 pad 29: SCL_2 -> TX
- U1 pad 3: Net-(U1-PC14) -> LED_7
- U1 pad 30: SDA_2 -> RX
- U1 pad 32: +3V0 -> VBAT
- U1 pad 35: IR_POW_4 -> LED_ESTADO
- U1 pad 36: IR_POW_3 -> ENABLE
- U1 pad 37: IR_POW_1 -> LED_R
- U1 pad 38: IR_POW_2 -> LED_G
- U1 pad 39: LED_1 -> LED_B
- U1 pad 4: Net-(U1-PC15) -> LED_6
- U1 pad 40: LED_2 -> PWM_FAN
- U1 pad 41: LED_R -> IN1_Der
- U1 pad 42: LED_G -> IN2_Der
- U1 pad 43: unconnected-(U1-PA10-Pad43) -> IN1_Izq
- U1 pad 44: CS -> IN2_Izq
- U1 pad 48: +3V0 -> VBAT
- U1 pad 50: LED_B -> CS
- U1 pad 51: LED_3 -> SCL
- U1 pad 52: LED_4 -> MISO
- U1 pad 53: unconnected-(U1-PC12-Pad53) -> MOSI
- U1 pad 54: IN1 -> unconnected-(U1-PD2-Pad54)
- U1 pad 55: SCL -> unconnected-(U1-PB3-Pad55)
- U1 pad 56: SDO/SA0 -> unconnected-(U1-PB4-Pad56)
- U1 pad 57: SDA -> unconnected-(U1-PB5-Pad57)
- U1 pad 6: RCC_OSC_OUT -> RCC_OSC_IN
- U1 pad 61: unconnected-(U1-PB8-Pad61) -> LED_10
- U1 pad 62: BUZZER_OP -> LED_9
- U1 pad 63: GND -> VSS
- U1 pad 64: +3V0 -> VBAT
- U1 pad 8: SEL -> IR_REC_4
- U1 pad 9: RUN -> IR_REC_1
- U3 pad 1: Net-(U3-BST) -> /AS5048_Izq/SDA_s
- U3 pad 2: GND -> /AS5048_Izq/SCL_s
- U3 pad 3: Net-(U3-FB) -> /AS5048_Izq/GND_s
- U3 pad 4: POW_IN -> /AS5048_Izq/GND_s
- U3 pad 5: POW_IN -> /AS5048_Izq/GND_s
- U3 pad 6: Net-(U3-SW) -> /AS5048_Izq/GND_s
- U4 pad 1: /AS5048_Izq/SDA_s -> /AS5048_Der/SDA_s
- U4 pad 11: /AS5048_Izq/+3V0_s -> /AS5048_Der/+3V0_s
- U4 pad 12: /AS5048_Izq/+3V0_s -> /AS5048_Der/+3V0_s
- U4 pad 13: /AS5048_Izq/GND_s -> /AS5048_Der/GND_s
- U4 pad 2: /AS5048_Izq/SCL_s -> /AS5048_Der/SCL_s
- U4 pad 3: /AS5048_Izq/GND_s -> /AS5048_Der/GND_s
- U4 pad 4: /AS5048_Izq/GND_s -> /AS5048_Der/+3V0_s
- U4 pad 5: /AS5048_Izq/GND_s -> /AS5048_Der/GND_s
- U4 pad 6: unconnected-(U4-TEST_6-Pad6) -> /AS5048_Der/GND_s
- U6 pad 1: SDO/SA0 -> /MP6551_Izq/SHUNT_MI
- U6 pad 10: unconnected-(U6-OCS_AUX-Pad10) -> /MP6551_Izq/SHUNT_MI
- U6 pad 12: CS -> unconnected-(U6-NFAULT-Pad12)
- U6 pad 13: SCL -> IN1_Izq
- U6 pad 14: SDA -> ENABLE
- U6 pad 2: GND -> POW_IN
- U6 pad 3: GND -> Net-(M2-+)
- U6 pad 4: unconnected-(U6-INT1-Pad4) -> ENABLE
- U6 pad 5: +3V0 -> IN2_Izq
- U6 pad 6: GND -> Net-(U6-SR)
- U6 pad 7: GND -> unconnected-(U6-CM2-Pad7)
- U6 pad 8: +3V0 -> Net-(M2-+)
- U6 pad 9: unconnected-(U6-INT2-Pad9) -> VSS
- Y1 pad 1: Net-(U1-PC14) -> RCC_OSC_IN
- Y1 pad 2: Net-(U1-PC15) -> VSS
Routing:
- net +3V0: track 122.3 -> 0.00 mm, vias 5 -> 0
- net SEL: track 66.3 -> 0.00 mm, vias 2 -> 0
- net NRST: track 54.0 -> 0.00 mm, vias 2 -> 0
- net RUN: track 50.4 -> 0.00 mm, vias 2 -> 0
- net +3V0(BAT): track 43.2 -> 0.00 mm, vias 2 -> 0
- net BAT_VOL: track 38.5 -> 0.00 mm, vias 2 -> 0
- net POW_IN: track 37.9 -> 0.00 mm
- net 3V0A: track 24.9 -> 0.00 mm, vias 2 -> 0
- net Net-(U3-SW): track 24.5 -> 0.00 mm
- net SYS_JTCK-SWCLK: track 20.1 -> 0.00 mm, vias 2 -> 0
- net SEL_LED: track 18.1 -> 0.00 mm, vias 2 -> 0
- net +3V3(ST-LINK): track 17.0 -> 0.00 mm
- net Net-(U1-BOOT0): track 16.2 -> 0.00 mm
- net Net-(U1-VCAP_1): track 15.0 -> 0.00 mm, vias 2 -> 0
- net SYS_JTMS-SWDIO: track 14.9 -> 0.00 mm, vias 2 -> 0
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- added copper zone on B.Cu, net VSS
- added copper zone on F.Cu, net VSS
- removed copper zone on B.Cu, net GND
- removed copper zone on F.Cu, net GND
Other:
- board size 88.3 x 94 mm -> 70 x 94 mm

Commit message: Esquematico corregido del micromouse
Parts:
- removed the Q3 at (110.1, 83.8)
- moved Q3 104.2 mm to (126.7, 121.4)
- renumbered C42 to C41, C41 to C42, D12 to D11, D11 to D12, Q12 to Q3

Commit message: Chasis minisumo terminado
Parts:
- removed the C10 at (202.5, 116.0)
- removed the C14 at (208.7, 103.7)
- removed the C17 at (202.5, 119.9)
- removed the C20 at (202.5, 121.9)
- removed the C21 at (202.5, 123.9)
- removed the C24 at (202.5, 125.8)
- removed the C25 at (211.1, 102.0)
- removed the C29 at (202.5, 127.8)
- removed the C30 at (209.7, 126.9)
- removed the C34 at (205.7, 116.0)
- removed the C39 at (213.6, 102.0)
- removed C45, C55: 10uF, Capacitor_SMD:C_0805_2012Metric
- removed C46, C59, C60, C63, C64: 0.1uF, Capacitor_SMD:C_0201_0603Metric
- removed C56: 470uF, Capacitor_THT:CP_Radial_D6.3mm_P2.50mm
- removed C57, C58, C61, C62: 10uF, Capacitor_SMD:C_1206_3216Metric
- removed the C9 at (199.3, 127.8)
- removed D18, D19, D20, D21: SFH_4550, SFH4550:DIO_SFH_4550
- removed IC2, IC3: AD8418AWHRZ, AD8418AWHRZ:SOIC127P600X175-8N
- removed J10: AS5048_Der, MicromouseHuellas:Encoder1
- removed Q10, Q11, Q6, Q7: SFH_309FA, SFH309FA:XDCR_SFH_309-4_5
- removed Q4, Q5, Q8, Q9: AO3400A, Package_TO_SOT_SMD:SOT-23
- removed R31, R32, R33, R34, R39, R40, R45, R46: 4.7k, Resistor_SMD:R_0201_0603Metric
- removed R41, R42, R47, R48: 30, Resistor_SMD:R_0805_2012Metric
- removed R43, R44, R49, R50: 1.5k, Resistor_SMD:R_0201_0603Metric
- removed the U3 at (229.9, 90.0)
- removed U4: AS5048B-HTSP, AS5048B-HTSP:SOP65P640X120-14N
- removed U5: LSM6DSRTR, LSM6DSRTR:PQFN50P250X300X86-14N
- added C11: 47uF, Capacitor_SMD:C_0805_2012Metric, F.Cu at (169.7, 126.7)
- added C12: 20pF, Capacitor_SMD:C_0402_1005Metric_Pad0.74x0.62mm_HandSolder, F.Cu at (114.2, 134.0)
- added C18: 10uF, Capacitor_SMD:C_0402_1005Metric_Pad0.74x0.62mm_HandSolder, F.Cu at (173.6, 126.2)
- added C19: 10uF, Capacitor_SMD:C_0402_1005Metric_Pad0.74x0.62mm_HandSolder, F.Cu at (173.6, 132.3)
- added C22: 10uF, Capacitor_SMD:C_0402_1005Metric_Pad0.74x0.62mm_HandSolder, F.Cu at (173.6, 128.7)
- added C23: 20pF, Capacitor_SMD:C_0402_1005Metric_Pad0.74x0.62mm_HandSolder, F.Cu at (116.3, 128.1)
- added C26: 10uF, Capacitor_SMD:C_0402_1005Metric_Pad0.74x0.62mm_HandSolder, F.Cu at (173.6, 131.1)
- added C28: 47uF, Capacitor_SMD:C_0805_2012Metric, F.Cu at (169.7, 131.9)
- added C32: 0.1uF, Capacitor_SMD:C_0402_1005Metric_Pad0.74x0.62mm_HandSolder, F.Cu at (173.6, 127.5)
- added C35: 0.1uF, Capacitor_SMD:C_0402_1005Metric_Pad0.74x0.62mm_HandSolder, F.Cu at (173.6, 129.9)
- added G***: LOGO, Imágenes:NINLogo, B.Cu at (146.3, 62.3)
- added G***: LOGO, Imágenes:DillingerLogo, B.Cu at (146.2, 117.6)
- added G***: LOGO, Imágenes:RobotronicsLogo, B.Cu at (146.2, 133.4)
- added J1: AS5048_Izq, MicromouseHuellas:ENCODER_PAD_PADRE, F.Cu at (113.5, 120.9)
- added J12: MOT_I, JST_SH_2PIN_SMD_VERTICAL:JST_BM02B-SRSS-TB_LF__SN_, F.Cu at (128.4, 96.9)
- added J13: MOT_D, JST_SH_2PIN_SMD_VERTICAL:JST_BM02B-SRSS-TB_LF__SN_, F.Cu at (165.4, 96.4)
- added J2: AS5048_Der, MicromouseHuellas:ENCODER_PAD_PADRE, F.Cu at (178.8, 120.9)
- added J3: MOT_FAN, JST_SH_2PIN_SMD_VERTICAL:JST_BM02B-SRSS-TB_LF__SN_, F.Cu at (141.6, 100.2)
- added J4: IR_LAT_Der, MicromouseHuellas:IR_SENSOR_2, F.Cu at (129.5, 62.6)
- added J5: IR_LAT_Izq, MicromouseHuellas:IR_SENSOR_2, F.Cu at (162.9, 62.6)
- added J7: IR_FRONT_Der, MicromouseHuellas:IR_SENSOR_2, F.Cu at (174.6, 85.9)
- added U10: AD8418AWHRZ, AD8418AWHRZ:SOIC127P600X175-8N, F.Cu at (151.7, 117.8)
- added U8: AD8418AWHRZ, AD8418AWHRZ:SOIC127P600X175-8N, F.Cu at (140.7, 117.8)
- added U9: MP6551GQB-Z, MP6551GQB-Z:MP6551GQBZ, F.Cu at (151.7, 111.3)
- C1: value 2.2uF -> 0.1uF; footprint Capacitor_SMD:C_0805_2012Metric -> Capacitor_SMD:C_0402_1005Metric_Pad0.74x0.62mm_HandSolder
- C14: renamed from C16; footprint Capacitor_SMD:C_0201_0603Metric -> Capacitor_SMD:C_0402_1005Metric_Pad0.74x0.62mm_HandSolder
- C15: value 47uF -> 10uF; footprint Capacitor_SMD:C_0805_2012Metric -> Capacitor_SMD:C_0402_1005Metric_Pad0.74x0.62mm_HandSolder
- C16: renamed from C18; footprint Capacitor_SMD:C_0201_0603Metric -> Capacitor_SMD:C_0402_1005Metric_Pad0.74x0.62mm_HandSolder
- C17: renamed from C19; footprint Capacitor_SMD:C_0201_0603Metric -> Capacitor_SMD:C_0402_1005Metric_Pad0.74x0.62mm_HandSolder
- C2: value 0.1uF -> 1uF
- C20: renamed from C22; footprint Capacitor_SMD:C_0201_0603Metric -> Capacitor_SMD:C_0402_1005Metric_Pad0.74x0.62mm_HandSolder
- C21: renamed from C23; footprint Capacitor_SMD:C_0201_0603Metric -> Capacitor_SMD:C_0402_1005Metric_Pad0.74x0.62mm_HandSolder
- C24: renamed from C26; footprint Capacitor_SMD:C_0201_0603Metric -> Capacitor_SMD:C_0402_1005Metric_Pad0.74x0.62mm_HandSolder
- C25: renamed from C27; footprint Capacitor_SMD:C_0201_0603Metric -> Capacitor_SMD:C_0402_1005Metric_Pad0.74x0.62mm_HandSolder
- C27: renamed from C28; value 0.01uF -> 10nF
- C29: renamed from C31; footprint Capacitor_SMD:C_0201_0603Metric -> Capacitor_SMD:C_0402_1005Metric_Pad0.74x0.62mm_HandSolder
- C3: footprint Capacitor_SMD:C_0805_2012Metric -> Capacitor_SMD:C_0402_1005Metric_Pad0.74x0.62mm_HandSolder
- C30: renamed from C32; footprint Capacitor_SMD:C_0201_0603Metric -> Capacitor_SMD:C_0402_1005Metric_Pad0.74x0.62mm_HandSolder
- C31: renamed from C33; footprint Capacitor_SMD:C_0201_0603Metric -> Capacitor_SMD:C_0402_1005Metric_Pad0.74x0.62mm_HandSolder
- C33: renamed from C35; footprint Capacitor_SMD:C_1206_3216Metric -> Capacitor_SMD:C_0402_1005Metric_Pad0.74x0.62mm_HandSolder
- C34: renamed from C36; footprint Capacitor_SMD:C_1206_3216Metric -> Capacitor_SMD:C_0402_1005Metric_Pad0.74x0.62mm_HandSolder
- C39: renamed from C41; footprint Capacitor_SMD:C_1206_3216Metric -> Capacitor_SMD:C_0805_2012Metric
- C4: value 0.1uF -> 2.2uF
- C41: renamed from C43; footprint Capacitor_SMD:C_1206_3216Metric -> Capacitor_SMD:C_0805_2012Metric
- C42: renamed from C44; footprint Capacitor_SMD:C_0201_0603Metric -> Capacitor_SMD:C_0402_1005Metric_Pad0.74x0.62mm_HandSolder
- C47: value 10uF -> 0.1uF; footprint Capacitor_SMD:C_0805_2012Metric -> Capacitor_SMD:C_0402_1005Metric_Pad0.74x0.62mm_HandSolder; moved to B.Cu
- C48: footprint Capacitor_SMD:C_0201_0603Metric -> Capacitor_SMD:C_0402_1005Metric_Pad0.74x0.62mm_HandSolder; moved to B.Cu
- C49: value 100nF -> 0.1uF; footprint Capacitor_SMD:C_0201_0603Metric -> Capacitor_SMD:C_0402_1005Metric_Pad0.74x0.62mm_HandSolder
- C50: value 100nF -> 10uF; footprint Capacitor_SMD:C_0201_0603Metric -> Capacitor_SMD:C_0402_1005Metric_Pad0.74x0.62mm_HandSolder
- C51, C54: value 100nF -> APV0609471M010R; footprint Capacitor_SMD:C_0201_0603Metric -> APV0609471M010R:CAPAE660X980N
- C52: value 10uF -> 0.1uF; footprint Capacitor_SMD:C_0805_2012Metric -> Capacitor_SMD:C_0402_1005Metric_Pad0.74x0.62mm_HandSolder
- C53: value 470uF -> 10uF; footprint Capacitor_THT:CP_Radial_D6.3mm_P2.50mm -> Capacitor_SMD:C_0402_1005Metric_Pad0.74x0.62mm_HandSolder
- C6: value 1uF -> 4.7uF
- C8: value 4.7uF -> 0.1uF
- C9: renamed from C11; footprint Capacitor_SMD:C_0201_0603Metric -> Capacitor_SMD:C_0402_1005Metric_Pad0.74x0.62mm_HandSolder
- J8: value Lipo -> IR_FRONT_Izq; footprint B2B-PH-SM4-TB_LF__SN:B2B-PH-SM4-TB_LF__SN_ -> MicromouseHuellas:IR_SENSOR_2
- J9: value AS5048_Izq -> Lipo; footprint MicromouseHuellas:Encoder1 -> Connector_PinHeader_2.54mm:PinHeader_1x02_P2.54mm_Vertical_SMD_Pin1Left
- L1: value CVH201610A-2R2M -> BMRA000404202R2MA1; footprint CVH201610A-2R2M:INDC2016X100N -> BMRA000404202R2MA1:BMRA000404202R2MA1
- R10: footprint Resistor_SMD:R_0402_1005Metric_Pad0.72x0.64mm_HandSolder -> Resistor_SMD:R_0805_2012Metric
- R16: value 1K -> 330
- R18, R22, R35, R37, R6: footprint Resistor_SMD:R_0201_0603Metric -> Resistor_SMD:R_0402_1005Metric_Pad0.72x0.64mm_HandSolder
- R19: value 82 -> 330; footprint Resistor_SMD:R_0201_0603Metric -> Resistor_SMD:R_0402_1005Metric_Pad0.72x0.64mm_HandSolder
- R20: value 10 -> 330; footprint Resistor_SMD:R_0201_0603Metric -> Resistor_SMD:R_0402_1005Metric_Pad0.72x0.64mm_HandSolder
- R21: value 22 -> 330; footprint Resistor_SMD:R_0201_0603Metric -> Resistor_SMD:R_0402_1005Metric_Pad0.72x0.64mm_HandSolder
- R4: footprint Resistor_SMD:R_0201_0603Metric -> Resistor_SMD:R_0805_2012Metric
- S2: value ButtonNRST -> BTN_NRST; footprint PTS636_SM43J_SMTR_LFS:SW_PTS636_SM43J_SMTR_LFS -> B3U-1000PM:SW_B3U-1000PM
- S3, S4, S5: footprint PTS636_SM43J_SMTR_LFS:SW_PTS636_SM43J_SMTR_LFS -> B3U-1000PM:SW_B3U-1000PM
- U6: value MP6551GQB-Z -> LSM6DSRTR; footprint MP6551GQB-Z:MP6551GQBZ -> LSM6DSRTR:PQFN50P250X300X86-14N; moved to B.Cu
- moved LS1 117.0 mm to (114.3, 138.1)
- moved D1 110.3 mm to (114.0, 141.9)
- moved Y1 110.0 mm to (113.9, 131.2), turned to 90 degrees
- moved Q1 103.6 mm to (119.3, 139.8), turned to 90 degrees
- moved C51 102.3 mm to (135.0, 99.9), turned to 90 degrees
- moved R5 99.7 mm to (117.8, 138.4)
- moved R35 97.9 mm to (137.2, 110.3), turned to 90 degrees
- moved R36 93.2 mm to (131.6, 110.9), turned to 180 degrees
- moved R1 93.2 mm to (121.9, 124.1)
- moved J8 90.4 mm to (117.7, 85.9), turned to -173 degrees
- moved C48 90.1 mm to (145.6, 104.9), turned to 180 degrees
- moved C15 89.3 mm to (122.0, 140.2), turned to 90 degrees
- moved U6 88.3 mm to (146.2, 102.5), turned to 180 degrees
- moved FB1 87.8 mm to (133.0, 140.4), turned to -90 degrees
- moved C1 87.2 mm to (126.2, 140.2), turned to 90 degrees
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- renumbered C12 to C10, C38 to C36, C40 to C38, C42 to C40, J5 to J6, IC1 to U3
Connections:
- C1 pad 1: Net-(U1-VCAP_1) -> GND
- C1 pad 2: VSS -> +3V0
- C10 pad 2: VSS -> GND
- C13 pad 1: VSS -> GND
- C14 pad 1: VBAT -> +3V0
- C14 pad 2: VSS -> GND
- C15 pad 1: VSS -> GND
- C15 pad 2: POW_IN -> +3V0
- C16 pad 1: VBAT -> +3V0
- C16 pad 2: VSS -> GND
- C17 pad 2: VSS -> GND
- C2 pad 1: VSS -> GND
- C2 pad 2: VBAT -> +3V0
- C20 pad 1: VBAT -> +3V0
- C20 pad 2: VSS -> GND
- C21 pad 2: VSS -> GND
- C24 pad 1: VBAT -> +3V0
- C24 pad 2: VSS -> GND
- C25 pad 2: VSS -> GND
- C27 pad 1: VBAT -> VDDA
- C27 pad 2: VSS -> GND
- C29 pad 1: VBAT -> +3V0
- C29 pad 2: VSS -> GND
- C3 pad 1: Net-(U1-VCAP_2) -> Net-(U1-VCAP_1)
- C3 pad 2: VSS -> GND
- C30 pad 2: VSS -> GND
- C31 pad 1: VBAT -> VDDA
- C31 pad 2: VSS -> GND
- C33 pad 1: VBAT -> +3V0
- C33 pad 2: VSS -> GND
- C34 pad 2: VSS -> GND
- C36 pad 2: VSS -> GND
- C37 pad 1: VSS -> NRST
- C37 pad 2: POW_IN -> GND
- C4 pad 1: VSS -> Net-(U1-VCAP_2)
- C4 pad 2: VBAT -> GND
- C40 pad 1: VBAT -> +3V0
- C40 pad 2: VSS -> GND
- C41 pad 2: VSS -> GND
- C42 pad 2: VSS -> GND
- C47 pad 1: /AS5048_Der/+3V0_s -> GND
- C47 pad 2: /AS5048_Der/GND_s -> +3V0
- C48 pad 1: /AS5048_Der/+3V0_s -> GND
- C48 pad 2: /AS5048_Der/GND_s -> +3V0
- C49 pad 1: VSS -> GND
- C49 pad 2: VBAT -> POW_IN
- C5 pad 1: VSS -> GND
- C5 pad 2: VBAT -> +3V0
- C50 pad 1: VSS -> GND
- C50 pad 2: VBAT -> POW_IN
- C51 pad 1: VSS -> POW_IN
- C51 pad 2: POW_IN -> GND
- C52 pad 1: VSS -> GND
- C53 pad 1: POW_IN -> GND
- C53 pad 2: VSS -> POW_IN
- C54 pad 1: VSS -> POW_IN
- C54 pad 2: POW_IN -> GND
- C6 pad 1: VSS -> GND
- C6 pad 2: VBAT -> +3V0
- C7 pad 1: VSS -> GND
- C7 pad 2: VBAT -> +3V0
- C8 pad 1: VSS -> GND
- C8 pad 2: VBAT -> +3V0
- C9 pad 1: VBAT -> +3V0
- C9 pad 2: VSS -> GND
- D1 pad C: VBAT -> +3V0
- D10 pad A: VSS -> GND
- D11 pad 1: VSS -> GND
- D11 pad 2: VSS -> GND
- D11 pad 3: VSS -> GND
- D12 pad C: VBAT -> +3V0
- D13 pad 1: VSS -> GND
- D14 pad 1: VSS -> GND
- D15 pad 1: VSS -> GND
- D16 pad 1: VSS -> GND
- D17 pad 1: VSS -> GND
- D3 pad 1: VSS -> GND
- D4 pad 1: VSS -> GND
- D5 pad 1: VSS -> GND
- D6 pad 1: VSS -> GND
- D7 pad 1: VSS -> GND
- D8 pad 1: VSS -> GND
- D9 pad 1: VSS -> GND
- FB1 pad 1: VBAT -> +3V0
- FB1 pad 2: VBAT -> VDDA
- J6 pad 4: VSS -> GND
- J8 pad 1: LIPO -> +3V0
- J8 pad 2: VSS -> IR_POW_4
- J8 pad 3: (no net) -> IR_REC_4
- J8 pad 4: (no net) -> GND
- J9 pad 1: /AS5048_Izq/+3V0_s -> LIPO
- J9 pad 2: /AS5048_Izq/SDA_s -> GND
- LS1 pad 1: VBAT -> +3V0
- Q1 pad 2: VSS -> GND
- Q2 pad 2: VSS -> GND
- Q3 pad 4: VSS -> GND
- R1 pad 1: VSS -> GND
- R16 pad 1: +3V3 -> +3V0
- R17 pad 1: VSS -> GND
- R18 pad 2: VSS -> GND
- R28 pad 1: VBAT -> +3V0
- R29 pad 1: VBAT -> +3V0
- R3 pad 2: VSS -> GND
- R30 pad 1: VBAT -> +3V0
- R35 pad 1: VSS -> GND
- R35 pad 2: Net-(U6-SR) -> Net-(U7-SR)
- R37 pad 1: VSS -> GND
- R37 pad 2: Net-(U7-SR) -> Net-(U9-SR)
- R38 pad 1: /MP6551_Der/SHUNT_MI -> /MP6551_Der/SHUNT_MD
- R5 pad 1: VSS -> GND
- R6 pad 1: VSS -> GND
- R7 pad 2: VSS -> GND
- R9 pad 1: VBAT -> +3V0
- S1 pad P$2: VSS -> GND
- S2 pad 2: VSS -> GND
- U1 pad 1: VBAT -> +3V0
- U1 pad 12: VSS -> GND
- U1 pad 13: VBAT -> VDDA
- U1 pad 18: VSS -> GND
- U1 pad 19: VBAT -> +3V0
- U1 pad 3: LED_7 -> LED_9
- U1 pad 32: VBAT -> +3V0
- U1 pad 4: LED_6 -> LED_10
- U1 pad 48: VBAT -> +3V0
- U1 pad 6: RCC_OSC_IN -> RCC_OSC_OUT
- U1 pad 61: LED_10 -> LED_6
- U1 pad 62: LED_9 -> LED_7
- U1 pad 63: VSS -> GND
- U1 pad 64: VBAT -> +3V0
- U2 pad 2: VSS -> GND
- U3 pad 2: VSS -> GND
- U3 pad 5: VBAT -> +3V0
- U6 pad 1: /MP6551_Izq/SHUNT_MI -> MISO
- U6 pad 10: /MP6551_Izq/SHUNT_MI -> unconnected-(U6-OCS_AUX-Pad10)
- U6 pad 12: unconnected-(U6-NFAULT-Pad12) -> CS
- U6 pad 13: IN1_Izq -> SCL
- U6 pad 14: ENABLE -> MOSI
- U6 pad 2: POW_IN -> GND
- U6 pad 3: Net-(M2-+) -> GND
- U6 pad 4: ENABLE -> unconnected-(U6-INT1-Pad4)
- U6 pad 5: IN2_Izq -> +3V0
- U6 pad 6: Net-(U6-SR) -> GND
- U6 pad 7: unconnected-(U6-CM2-Pad7) -> GND
- U6 pad 8: Net-(M2-+) -> +3V0
- U6 pad 9: VSS -> unconnected-(U6-INT2-Pad9)
- U7 pad 1: Net-(M3--) -> /MP6551_Izq/SHUNT_MI
- U7 pad 10: Net-(M3--) -> /MP6551_Izq/SHUNT_MI
- U7 pad 13: IN1_Der -> IN1_Izq
- U7 pad 3: /MP6551_Der/SHUNT_MI -> /MP6551_Izq/MOT_I+
- U7 pad 5: IN2_Der -> IN2_Izq
- U7 pad 8: /MP6551_Der/SHUNT_MI -> /MP6551_Izq/MOT_I+
- U7 pad 9: VSS -> GND
- Y1 pad 1: RCC_OSC_IN -> RCC_OSC_OUT
- Y1 pad 2: VSS -> GND
- Y1 pad 3: RCC_OSC_OUT -> RCC_OSC_IN
- Y1 pad 4: VSS -> GND
Routing:
- net +3V0: track 0.00 -> 483.9 mm, vias 0 -> 7
- net IR_REC_3: track 0.00 -> 177.1 mm, vias 0 -> 3
- net CURRENT_MI: track 0.00 -> 144.5 mm, vias 0 -> 2
- net IR_POW_3: track 0.00 -> 140.3 mm, vias 0 -> 2
- net POW_IN: track 0.00 -> 134.2 mm, vias 0 -> 23
- net CURRENT_MD: track 0.00 -> 134.0 mm, vias 0 -> 2
- net IR_REC_2: track 0.00 -> 127.3 mm, vias 0 -> 3
- net SCL_s: track 0.00 -> 124.6 mm, vias 0 -> 4
- net SDA_s: track 0.00 -> 122.2 mm, vias 0 -> 4
- net LED_R: track 0.00 -> 120.5 mm, vias 0 -> 2
- net IR_POW_2: track 0.00 -> 116.5 mm, vias 0 -> 2
- net LED_G: track 0.00 -> 113.1 mm, vias 0 -> 2
- net LED_B: track 0.00 -> 106.8 mm, vias 0 -> 2
- net ENABLE: track 0.00 -> 104.1 mm, vias 0 -> 4
- net IR_POW_1: track 0.00 -> 89.3 mm, vias 0 -> 2
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- added copper zone on B.Cu, net +5V
- added copper zone on F.Cu, net +5V
- added copper zone on B.Cu, net /MP6551_Der/MOT_D-
- added copper zone on F.Cu, net /MP6551_Der/MOT_D-
- added copper zone on B.Cu, net /MP6551_Der/SHUNT_MD
- added copper zone on F.Cu, net /MP6551_Der/SHUNT_MD
- added copper zone on B.Cu, net /MP6551_Izq/MOT_I+
- added copper zone on F.Cu, net /MP6551_Izq/MOT_I+
- added copper zone on B.Cu, net /MP6551_Izq/SHUNT_MI
- added copper zone on F.Cu, net /MP6551_Izq/SHUNT_MI
- added copper zone on B.Cu, net GND
- added copper zone on F.Cu, net GND
- added copper zone on B.Cu, net LIPO
- added copper zone on F.Cu, net LIPO
- added copper zone on B.Cu, net POW_IN
- added copper zone on F.Cu, net POW_IN
- removed copper zone on B.Cu, net VSS
- removed copper zone on F.Cu, net VSS
Other:
- board size 70 x 94 mm -> 70 x 92 mm
- board text added: "+ -"

Commit message: Red 3V0 cambiada a 3V3
Parts:
- C10: value 0.1uf -> 0.1uF
- U3: value ME6211C30M5G -> ME6211C33M5G
Connections:
- net +3V0 renamed +3V3
