File: Micromouse/Micromouse.kicad_sch (KiCad schematic)
At the start: 68 parts, among them J1 ST-LINK, J2 AS5048_Izq, J3 AS5048_Der, J4 IR_1, J5 IR_2, J6 IR_3, J7 IR_4, J8 Lipo, Q1 AO3400A, U1 STM32F405RGTx, U2 MP2359DJ-LF-Z, Y1 32.768kHz, Y2 25MHz

Commit message: Commit4
Parts:
- removed BZ1: Buzzer, Buzzer_Beeper:Buzzer_TDK_PS1240P02BT_D12.2mm_H6.5mm, symbol Device:Buzzer
- removed C1, C3: 12.5pF, Capacitor_SMD:C_0201_0603Metric, symbol Device:C
- removed D2: LED, LED_SMD:LED_0201_0603Metric, symbol Device:LED
- removed J1: ST-LINK, S4B-XH-SM4-TB:JST_S4B-XH-SM4-TB, symbol S4B-XH-SM4-TB:S4B-XH-SM4-TB
- removed S1: ButtonS, PTS636_SM43J_SMTR_LFS:SW_PTS636_SM43J_SMTR_LFS, symbol PTS636_SM43J_SMTR_LFS:PTS636_SM43J_SMTR_LFS
- removed S2: CUS-12TB, CUS-12TB:CUS-12B, symbol CUS-12TB:CUS-12TB
- removed Y1: 32.768kHz, CC5V-T1A_32.768KHZ_12.5PF_20PPM_TA_QC:XTAL_CC5V-T1A_32.768KHZ_12.5PF_20PPM_TA_QC, symbol CC5V-T1A_32.768KHZ_12.5PF_20PPM_TA_QC:CC5V-T1A_32.768KHZ_12.5PF_20PPM_TA_QC
- removed Y2: 25MHz, Crystal25MHz:XTAL_C3E-25.000-12-3030-X-R, symbol C3E-25.000-12-3030-X-R:C3E-25.000-12-3030-X-R
- added C12: 0.1uf, Capacitor_SMD:C_0402_1005Metric_Pad0.74x0.62mm_HandSolder, symbol Device:C
- added C13, C15, C30: 47uF, Capacitor_SMD:C_0805_2012Metric, symbol Device:C
- added C17, C20, C21, C24, C29, C41: 10uF, Capacitor_SMD:C_0402_1005Metric_Pad0.74x0.62mm_HandSolder, symbol Device:C
- added C19, C23, C27, C32: 10uF, Capacitor_SMD:C_0201_0603Metric, symbol Device:C
- added C2, C34, C37, C4, C5, C7, C9: 0.1uF, Capacitor_SMD:C_0402_1005Metric_Pad0.74x0.62mm_HandSolder, symbol Device:C
- added C36: 10uF, Capacitor_SMD:C_1206_3216Metric, symbol Device:C
- added C38: 1uF, Capacitor_SMD:C_0402_1005Metric_Pad0.74x0.62mm_HandSolder, symbol Device:C
- added C8: 4.7uF, Capacitor_SMD:C_0402_1005Metric_Pad0.74x0.62mm_HandSolder, symbol Device:C
- added D13, D14, D15, D16, D17, D6, D9: LED, LED_SMD:LED_0805_2012Metric, symbol Device:LED
- added D2: 1N5819HW-7, 1N5819HW-7:SOD3715X145N, symbol 1N5819HW-7:1N5819HW-7
- added IC1: ME6211C30M5G, ME6211C33M5G:SOT95P282X145-5N, symbol ME6211C33M5G:ME6211C33M5G
- added J5: ST_LINK, JST_SH_6PIN_SMD_HORIZONTAL:JST_SM06B-SRSS-TB_LF__SN_, symbol SM06B-SRSS-TB_LF__SN_:SM06B-SRSS-TB_LF__SN_
- added JP1: SolderJumper_2_Open, Jumper:SolderJumper-2_P1.3mm_Open_RoundedPad1.0x1.5mm, symbol Jumper:SolderJumper_2_Open
- added LS1: Buzzer, CMT-0502-03-SMT-TR:CMT050203SMTTR, symbol CMT-0502-03-SMT-TR:CMT-0502-03-SMT-TR
- added M1: MOT_FAN, symbol Motor Coreless:Motor_Coreless_Micromouse
- added Q12: AON7423, AON7423:AON7423, symbol AON7423:AON7423
- added Q2: AO3400A, Package_TO_SOT_SMD:SOT-23, symbol Transistor_FET:AO3400A
- added R15, R23, R24, R25, R26, R27: 330, Resistor_SMD:R_0402_1005Metric_Pad0.72x0.64mm_HandSolder, symbol Device:R
- added R16: 1K, Resistor_SMD:R_0402_1005Metric_Pad0.72x0.64mm_HandSolder, symbol Device:R
- added R17: 47K, Resistor_SMD:R_0402_1005Metric_Pad0.72x0.64mm_HandSolder, symbol Device:R
- added R28: 100K, Resistor_SMD:R_0402_1005Metric_Pad0.72x0.64mm_HandSolder, symbol Device:R
- added R29: 33K, Resistor_SMD:R_0402_1005Metric_Pad0.72x0.64mm_HandSolder, symbol Device:R
- added R3: 27K, Resistor_SMD:R_0402_1005Metric_Pad0.72x0.64mm_HandSolder, symbol Device:R
- added R30: 4.7K, Resistor_SMD:R_0402_1005Metric_Pad0.72x0.64mm_HandSolder, symbol Device:R
- added R4: 220, Resistor_SMD:R_0201_0603Metric, symbol Device:R
- added R6: 10k, Resistor_SMD:R_0201_0603Metric, symbol Device:R
- added S1: CUS-12TB, CUS-12TB:CUS-12B, symbol CUS-12TB:CUS-12TB
- added S3: BTN_1, PTS636_SM43J_SMTR_LFS:SW_PTS636_SM43J_SMTR_LFS, symbol PTS636_SM43J_SMTR_LFS:PTS636_SM43J_SMTR_LFS
- added S5: BTN_3, PTS636_SM43J_SMTR_LFS:SW_PTS636_SM43J_SMTR_LFS, symbol PTS636_SM43J_SMTR_LFS:PTS636_SM43J_SMTR_LFS
- added Y1: 8MHz, 8.000MHz3.2x2.5mm:XTAL_C3E-8.000-18-3030-R, symbol C3E-8.000-18-3030-R:C3E-8.000-18-3030-R
- C10, C6: value 0.1uF -> 1uF; footprint Capacitor_SMD:C_0201_0603Metric -> Capacitor_SMD:C_0402_1005Metric_Pad0.74x0.62mm_HandSolder
- D3, D4: footprint LED_SMD:LED_0201_0603Metric -> LED_SMD:LED_0402_1005Metric_Pad0.77x0.64mm_HandSolder
- D5: footprint LED_SMD:LED_0201_0603Metric -> LED_SMD:LED_0805_2012Metric
- D7, D8: footprint LED_SMD:LED_0805_2012Metric_Pad1.15x1.40mm_HandSolder -> LED_SMD:LED_0805_2012Metric
- J3: renamed from J4; value IR_1 -> IR_LAT_Der
- J4: renamed from J5; value IR_2 -> IR_LAT_Izq
- J6: value IR_3 -> IR_FRONT_Der
- J7: value IR_4 -> IR_FRONT_Izq
- R10, R11, R12: value 220 -> 330; footprint Resistor_SMD:R_0201_0603Metric -> Resistor_SMD:R_0402_1005Metric_Pad0.72x0.64mm_HandSolder
- R13: value 10k -> 330; footprint Resistor_SMD:R_0805_2012Metric -> Resistor_SMD:R_0402_1005Metric_Pad0.72x0.64mm_HandSolder
- R14: value 4.7k -> 330; footprint Resistor_SMD:R_0201_0603Metric -> Resistor_SMD:R_0402_1005Metric_Pad0.72x0.64mm_HandSolder
- R2: value 120 -> 47K; footprint Resistor_SMD:R_0805_2012Metric -> Resistor_SMD:R_0402_1005Metric_Pad0.72x0.64mm_HandSolder
- R22: renamed from R16; value 27k -> 51k
- R7: value 220 -> 1K; footprint Resistor_SMD:R_0201_0603Metric -> Resistor_SMD:R_0402_1005Metric_Pad0.72x0.64mm_HandSolder
- R8: value 220 -> 10K; footprint Resistor_SMD:R_0201_0603Metric -> Resistor_SMD:R_0402_1005Metric_Pad0.72x0.64mm_HandSolder
- R9: value 220 -> 47k; footprint Resistor_SMD:R_0201_0603Metric -> Resistor_SMD:R_0402_1005Metric_Pad0.72x0.64mm_HandSolder
- S4: value ButtonC -> BTN_2
- renumbered C2 to C1, C16 to C14, C5 to C16, C12 to C18, C13 to C22, C21 to C25, C14 to C26, C7 to C28, C4 to C3, C17 to C31, C8 to C33, C19 to C35, C9 to C39, C15 to C40, C18 to C42, C20 to C43, C22 to C44, D9 to D11, D6 to D12, J2 to J1, J3 to J2, R3 to R1, R15 to R18, R4 to R19, R5 to R20, R6 to R21, R1 to R5, S3 to S2
Connections:
- net 3V0A is gone; now on net +3V0: C28.1, C33.1, FB1.2, U1.13 (VDDA)
- net CM2 is gone; now on net LED_1: U1.24 (PC4)
- net EN1 is gone; now on net IR_POW_3: U1.17 (PA3)
- net EN2 is gone; now on net IR_REC_3: U1.11 (PC3)
- net IN2 is gone; now on net LED_2: U1.25 (PC5)
- net +3V0: now also C10.2, C6.2, D1.C, D11.C, R9.1, C17.2, C2.2, C4.2, C41.1, C5.2, C7.2, C8.2, C9.2, IC1.5 (VOUT), LS1.1 (+), R28.1, R29.1, R30.1; no longer D7.2 (A)
- net +3V3(ST-LINK): now also J5.1
- net BUZZER_OP: no longer U1.62 (PB9)
- net CS: now also U1.50 (PA15); no longer U1.44 (PA11)
- net GND: now also C10.1, C6.1, D3.1 (K), D4.1 (K), D5.1 (K), D7.1 (K), D8.1 (K), C12.2, C13.1, C15.1, C17.1, C19.2, C2.1, C20.1, C21.1, C23.2, C24.1, C27.2, C29.1, C30.1, C32.2, C34.1, C36.2, C37.1, C38.2, C4.1, C41.2, C5.1, C7.1, C8.1, C9.1, D13.1 (K), D14.1 (K), D15.1 (K), D16.1 (K), D17.1 (K), D6.1 (K), D9.1 (K), IC1.2 (VSS), J5.4, Q12.4 (G), Q2.2 (S), R17.1, R3.2, R6.1, S1.P$2 (2), Y1.2 (GND), Y1.4 (GND); no longer C10.2, C6.2, R10.2, R11.2, R12.1, R14.2, R8.2, R9.2, S4.2
- net IR_POW_1: now also U1.15 (PA1); no longer U1.37 (PC6)
- net IR_POW_2: now also U1.16 (PA2); no longer U1.38 (PC7)
- net IR_POW_3: no longer U1.36 (PB15)
- net IR_POW_4: now also U1.14 (PA0); no longer U1.35 (PB14)
- net IR_REC_1: now also U1.9 (PC1); no longer U1.15 (PA1)
- net IR_REC_2: now also U1.10 (PC2); no longer U1.20 (PA4)
- net IR_REC_3: no longer U1.21 (PA5)
- net IR_REC_4: now also U1.8 (PC0); no longer U1.23 (PA7)
- net LED_1: now also R11.1; no longer D5.2 (A), U1.39 (PC8)
- net LED_2: now also R12.1; no longer D4.2 (A), U1.40 (PC9)
- net LED_3: now also R13.1, U1.26 (PB0); no longer D3.2 (A), U1.51 (PC10)
- net LED_4: now also R14.1, U1.27 (PB1); no longer U1.52 (PC11)
- net LED_B: now also U1.39 (PC8); no longer U1.50 (PA15)
- net LED_G: now also U1.38 (PC7); no longer U1.42 (PA9)
- net LED_R: now also U1.37 (PC6); no longer U1.41 (PA8)
- net NRST: now also R9.2
- net POW_IN: now also R2.1, C13.2, C15.2, C20.2, C21.2, C24.2, C29.2, C30.2, C34.2, C37.2, D2.C, JP1.1 (A), M1.1 (+), Q12.5 (D_1), Q12.6 (D_2), Q12.7 (D_3), Q12.8 (D_4), Q12.9 (D_5); no longer J8.1, R13.1, R2.2
- net PWM_FAN: now also U1.40 (PC9), R4.2; no longer U1.16 (PA2)
- net RCC_OSC_IN: now also U1.6 (PH1), Y1.1
- net RCC_OSC_OUT: now also Y1.3; no longer U1.6 (PH1)
- net SCL: now also U1.51 (PC10); no longer U1.55 (PB3)
- net SYS_JTCK-SWCLK: now also J5.3
- net SYS_JTMS-SWDIO: now also J5.2
- net at D1.A, Q1.3 (D): now also LS1.2 (-)
- net LED_7: now reaches U1.3 (PC14)
- net LED_7: now also R24.1
- net LED_6: now reaches U1.4 (PC15)
- net LED_6: now also R23.1
- net LED_8: now reaches U1.2 (PC13)
- net LED_8: now also R25.1
- net IN1_Izq: now reaches U1.43 (PA10)
- net MOSI: now reaches U1.53 (PC12)
- net LED_10: now reaches U1.61 (PB8)
- net LED_10: now also R27.1
- net at R7.1: now also R8.1, S1.P$1 (1)
- net at R12.2: now also D6.2 (A); no longer D8.1 (K)
- net LED_ESTADO: now reaches R10.1
- net LED_ESTADO: now also U1.35 (PB14); no longer D5.1 (K)
- net +3V0(BAT) renamed +5V
- net +5V: now also C12.1, C19.1, C23.1, C27.1, C32.1, C36.1, IC1.1 (VIN), IC1.3 (CE)
- removed net BAT_VOL: R13.2, R14.1, U1.14 (PA0)
- net CM1 renamed CURRENT_MI
- net IN1: no longer names the net of U1.54 (PD2)
- net NFAULT renamed LED_5
- net LED_5: now also R15.1
- removed net RUN: C10.1, S4.1, U1.9 (PC1)
- net SCL_1 renamed SCL_s
- net SCL_s: now also J2.3 (Pin_3)
- net SCL_2 renamed TX
- net TX: now also J5.5; no longer J2.3 (Pin_3)
- net SDA: no longer names the net of U1.57 (PB5)
- net SDA_1 renamed SDA_s
- net SDA_s: now also J2.2 (Pin_2)
- net SDA_2 renamed RX
- net RX: now also J5.6; no longer J2.2 (Pin_2)
- net SDO/SA0: no longer names the net of U1.56 (PB4)
- removed net SEL: C6.1, U1.8 (PC0)
- net SEL_LED: no longer names the net of D8.2 (A)
- net SEL_LED: now also R14.2; no longer U1.10 (PC2)
- new net: D13.2 (A), R23.2
- new net: R28.2, S3.2
- new net: D16.2 (A), R26.2
- new net: D14.2 (A), R24.2
- new net: D17.2 (A), R27.2
- new net: D4.2 (A), R16.2
- new net: D7.2 (A), R13.2
- new net: D15.2 (A), R25.2
- new net: D5.2 (A), R11.2
- new net: D3.2 (A), R10.2
- new net: J5.S1 (SHIELD), J5.S2 (SHIELD)
- new net: D2.A, M1.2 (-), Q2.3 (D)
- new net: D9.2 (A), R15.2
- new net: R29.2, S4.2
- new net: R30.2, S5.2
- new net: Q2.1 (G), R4.1, R6.2
- new net +3V3: R16.1
- new net BAT_VOLTAGE: R2.2, R3.1, U1.20 (PA4)
- new net CURRENT_MD: U1.21 (PA5)
- new net ENABLE: U1.36 (PB15)
- new net IN1_Der: U1.41 (PA8)
- new net IN2_Der: U1.42 (PA9)
- new net IN2_Izq: U1.44 (PA11)
- new net LED_9: R26.1, U1.62 (PB9)
- new net LIPO: C38.1, J8.1, JP1.2 (B), Q12.1 (S_1), Q12.2 (S_2), Q12.3 (S_3), R8.2
- new net MENU_ESTADO: R17.2, S3.1, S4.1, S5.1, U1.23 (PA7)
- new net MISO: U1.52 (PC11)
- no-connect marks 13 -> 12
Other:
- sheet MP6551 renamed MP6551_Izq
- removed sheet Fan
- added sheet MP6551_Der (MP6551_Der.kicad_sch)
- sheet LSM6DSRTR: file MPU6500.kicad_sch -> LSM6DSRTR.kicad_sch
- sheet LSM6DSRTR ports: added MISO, MOSI; removed SDA, SDO/SA0
- sheet MP6551_Izq: file DRV8833.kicad_sch -> MP6551_Izq.kicad_sch
- sheet MP6551_Izq ports: added CURRENT_MI, ENABLE, IN1_Izq, IN2_Izq; removed CM1, CM2, EN1, EN2, IN1, IN2, NFAULT
- note added: "Circuito de la turbina"
- note added: "Comunicación ST-LINK V3"
- note added: "Leds y botones de selección"
- note added: "Pads de conexión"
- note removed: "Botón de confirmacíón"
- note removed: "Botón de selección"
- note removed: "Led de selección"
- note removed: "Leds de estado"
- note removed: "Pines y pads"
- moved on the sheet: C1, C11, C14, C16, C18, C22, C25, C26, C28, C3, C31, C33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

Commit message: Esquematico corregido del micromouse
Parts:
- renumbered C42 to C41, C41 to C42, D12 to D11, D11 to D12, Q12 to Q3
Changed lines of the file:
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@@
 		(on_board yes)
 		(dnp no)
-		(property "Reference" "#PWR045"
+		(property "Reference" "#PWR046"
 			(at 346.075 92.583 0)
 			(effects
@@
 			(project "Micromouse"
 				(path "/96b72c82-8e98-4b00-820e-849de0fa96c7"
-					(reference "#PWR045")
+					(reference "#PWR046")
 					(unit 1)
 				)
@@
 		(dnp no)
 		(fields_autoplaced yes)
-		(property "Reference" "#PWR072"
+		(property "Reference" "#PWR041"
 			(at 305.308 85.09 0)
 			(effects
@@
 			(project "Micromouse"
 				(path "/96b72c82-8e98-4b00-820e-849de0fa96c7"
-					(reference "#PWR072")
+					(reference "#PWR041")
 					(unit 1)
 				)
@@
 		(dnp no)
 		(fields_autoplaced yes)
-		(property "Reference" "Q12"
+		(property "Reference" "Q3"
 			(at 327.914 61.214 0)
 			(effects
@@
 			(project ""
 				(path "/96b72c82-8e98-4b00-820e-849de0fa96c7"
-					(reference "Q12")
+					(reference "Q3")
 					(unit 1)
 				)
@@
 		(on_board yes)
 		(dnp no)
-		(property "Reference" "#PWR049"
+		(property "Reference" "#PWR050"
 			(at 355.6 219.456 0)
 			(effects
@@
 			(project "Micromouse"
 				(path "/96b72c82-8e98-4b00-820e-849de0fa96c7"
-					(reference "#PWR049")
+					(reference "#PWR050")
 					(unit 1)
 				)
@@
 		(on_board yes)
 		(dnp no)
-		(property "Reference" "#PWR044"
+		(property "Reference" "#PWR045"
 			(at 338.074 237.744 0)
 			(effects
@@
 			(project "Micromouse"
 				(path "/96b72c82-8e98-4b00-820e-849de0fa96c7"
-					(reference "#PWR044")
+					(reference "#PWR045")
 					(unit 1)
 				)
@@
 		(on_board yes)
 		(dnp no)
-		(property "Reference" "#PWR050"
+		(property "Reference" "#PWR051"
 			(at 384.81 95.758 0)
 			(effects
@@
 			(project "Micromouse"
 				(path "/96b72c82-8e98-4b00-820e-849de0fa96c7"
-					(reference "#PWR050")
+					(reference "#PWR051")
 					(unit 1)
 				)
@@
 		(on_board yes)
 		(dnp no)
-		(property "Reference" "#PWR043"
+		(property "Reference" "#PWR044"
 			(at 338.074 209.804 0)
 			(effects
@@
 			(project "Micromouse"
 				(path "/96b72c82-8e98-4b00-820e-849de0fa96c7"
-					(reference "#PWR043")
+					(reference "#PWR044")
 					(unit 1)
 				)
@@
 		(on_board yes)
 		(dnp no)
-		(property "Reference" "#PWR047"
+		(property "Reference" "#PWR048"
 			(at 350.266 159.258 0)
 			(effects
@@
 			(project "Micromouse"
 				(path "/96b72c82-8e98-4b00-820e-849de0fa96c7"
-					(reference "#PWR047")
+					(reference "#PWR048")
 					(unit 1)
 				)
@@
 		(dnp no)
 		(fields_autoplaced yes)
-		(property "Reference" "#PWR041"
+		(property "Reference" "#PWR042"
 			(at 308.229 173.99 0)
 			(effects
@@
 			(project "Micromouse"
 				(path "/96b72c82-8e98-4b00-820e-849de0fa96c7"
-					(reference "#PWR041")
+					(reference "#PWR042")
 					(unit 1)
 				)
@@
 		(on_board yes)
 		(dnp no)
-		(property "Reference" "D12"
+		(property "Reference" "D11"
 			(at 373.38 162.56 0)
 			(effects
@@
 			(project ""
 				(path "/96b72c82-8e98-4b00-820e-849de0fa96c7"
-					(reference "D12")
+					(reference "D11")
 					(unit 1)
 				)
@@
 		(on_board yes)
 		(dnp no)
-		(property "Reference" "#PWR052"
+		(property "Reference" "#PWR058"
 			(at 402.59 93.218 0)
 			(effects
@@
 			(project "Micromouse"
 				(path "/96b72c82-8e98-4b00-820e-849de0fa96c7"
-					(reference "#PWR052")
+					(reference "#PWR058")
 					(unit 1)
 				)
@@
 		(dnp no)
 		(fields_autoplaced yes)
-		(property "Reference" "#PWR048"
+		(property "Reference" "#PWR049"
 			(at 350.393 183.388 0)
 			(effects
@@
 			(project "Half-Size Micromouse"
 				(path "/96b72c82-8e98-4b00-820e-849de0fa96c7"
-					(reference "#PWR048")
+					(reference "#PWR049")
 					(unit 1)
 				)
@@
 		(on_board yes)
 		(dnp no)
-		(property "Reference" "#PWR051"
+		(property "Reference" "#PWR052"
 			(at 384.81 107.188 0)
 			(effects
@@
 			(project "Micromouse"
 				(path "/96b72c82-8e98-4b00-820e-849de0fa96c7"
-					(reference "#PWR051")
+					(reference "#PWR052")
 					(unit 1)
 				)
@@
 		(on_board yes)
 		(dnp no)
-		(property "Reference" "C42"
+		(property "Reference" "C41"
 			(at 385.318 59.69 0)
 			(effects
@@
 			(project "Half-Size Micromouse"
 				(path "/96b72c82-8e98-4b00-820e-849de0fa96c7"
-					(reference "C42")
+					(reference "C41")
 					(unit 1)
 				)
@@
 		(on_board yes)
 		(dnp no)
-		(property "Reference" "C41"
+		(property "Reference" "C42"
 			(at 380.492 94.488 0)
 			(effects
@@
 			(project "Micromouse"
 				(path "/96b72c82-8e98-4b00-820e-849de0fa96c7"
-					(reference "C41")
+					(reference "C42")
 					(unit 1)
 				)
@@
 		(on_board yes)
 		(dnp no)
-		(property "Reference" "D11"
+		(property "Reference" "D12"
 			(at 395.605 90.043 0)
 			(effects
@@
 			(project "Half-Size Micromouse"
 				(path "/96b72c82-8e98-4b00-820e-849de0fa96c7"
-					(reference "D11")
+					(reference "D12")
 					(unit 1)
 				)
@@
 		(on_board yes)
 		(dnp no)
-		(property "Reference" "#PWR042"
+		(property "Reference" "#PWR043"
 			(at 329.184 237.744 0)
 			(effects
@@
 			(project "Micromouse"
 				(path "/96b72c82-8e98-4b00-820e-849de0fa96c7"
-					(reference "#PWR042")
+					(reference "#PWR043")
 					(unit 1)
 				)
@@
 		(dnp no)
 		(fields_autoplaced yes)
-		(property "Reference" "#PWR046"
+		(property "Reference" "#PWR047"
 			(at 347.98 104.648 0)
 			(effects
@@
 			(project "Micromouse"
 				(path "/96b72c82-8e98-4b00-820e-849de0fa96c7"
-					(reference "#PWR046")
+					(reference "#PWR047")
 					(unit 1)
 				)

Commit message: Chasis minisumo terminado
Parts:
- removed C10: 1uF, Capacitor_SMD:C_0402_1005Metric_Pad0.74x0.62mm_HandSolder, symbol Device:C
- removed C9: 0.1uF, Capacitor_SMD:C_0402_1005Metric_Pad0.74x0.62mm_HandSolder, symbol Device:C
- removed L1: CVH201610A-2R2M, CVH201610A-2R2M:INDC2016X100N, symbol CVH201610A-2R2M:CVH201610A-2R2M
- removed M1: MOT_FAN, symbol Motor Coreless:Motor_Coreless_Micromouse
- removed S2: ButtonNRST, PTS636_SM43J_SMTR_LFS:SW_PTS636_SM43J_SMTR_LFS, symbol PTS636_SM43J_SMTR_LFS:PTS636_SM43J_SMTR_LFS
- removed S3: BTN_1, PTS636_SM43J_SMTR_LFS:SW_PTS636_SM43J_SMTR_LFS, symbol PTS636_SM43J_SMTR_LFS:PTS636_SM43J_SMTR_LFS
- removed S4: BTN_2, PTS636_SM43J_SMTR_LFS:SW_PTS636_SM43J_SMTR_LFS, symbol PTS636_SM43J_SMTR_LFS:PTS636_SM43J_SMTR_LFS
- removed S5: BTN_3, PTS636_SM43J_SMTR_LFS:SW_PTS636_SM43J_SMTR_LFS, symbol PTS636_SM43J_SMTR_LFS:PTS636_SM43J_SMTR_LFS
- added J3: MOT_FAN, JST_SH_2PIN_SMD_VERTICAL:JST_BM02B-SRSS-TB_LF__SN_, symbol BM02B-SRSS-TB_LF__SN_:BM02B-SRSS-TB_LF__SN_
- added L1: BMRA000404202R2MA1, BMRA000404202R2MA1, symbol BMRA000404202R2MA1:BMRA000404202R2MA1
- added S2: BTN_NRST, B3U-1000PM:SW_B3U-1000PM, symbol B3U-1000PM:B3U-1000PM
- added S3: BTN_1, B3U-1000PM:SW_B3U-1000PM, symbol B3U-1000PM:B3U-1000PM
- added S4: BTN_2, B3U-1000PM:SW_B3U-1000PM, symbol B3U-1000PM:B3U-1000PM
- added S5: BTN_3, B3U-1000PM:SW_B3U-1000PM, symbol B3U-1000PM:B3U-1000PM
- C10: renamed from C12; value 0.1uf -> 0.1uF
- C12: renamed from C14; footprint Capacitor_SMD:C_0201_0603Metric -> Capacitor_SMD:C_0402_1005Metric_Pad0.74x0.62mm_HandSolder
- C14: renamed from C16; footprint Capacitor_SMD:C_0201_0603Metric -> Capacitor_SMD:C_0402_1005Metric_Pad0.74x0.62mm_HandSolder
- C16: renamed from C18; footprint Capacitor_SMD:C_0201_0603Metric -> Capacitor_SMD:C_0402_1005Metric_Pad0.74x0.62mm_HandSolder
- C17: renamed from C19; footprint Capacitor_SMD:C_0201_0603Metric -> Capacitor_SMD:C_0402_1005Metric_Pad0.74x0.62mm_HandSolder
- C20: renamed from C22; footprint Capacitor_SMD:C_0201_0603Metric -> Capacitor_SMD:C_0402_1005Metric_Pad0.74x0.62mm_HandSolder
- C21: renamed from C23; footprint Capacitor_SMD:C_0201_0603Metric -> Capacitor_SMD:C_0402_1005Metric_Pad0.74x0.62mm_HandSolder
- C23: renamed from C25; footprint Capacitor_SMD:C_0201_0603Metric -> Capacitor_SMD:C_0402_1005Metric_Pad0.74x0.62mm_HandSolder
- C24: renamed from C26; footprint Capacitor_SMD:C_0201_0603Metric -> Capacitor_SMD:C_0402_1005Metric_Pad0.74x0.62mm_HandSolder
- C25: renamed from C27; footprint Capacitor_SMD:C_0201_0603Metric -> Capacitor_SMD:C_0402_1005Metric_Pad0.74x0.62mm_HandSolder
- C27: renamed from C28; value 0.01uF -> 10nF
- C29: renamed from C31; footprint Capacitor_SMD:C_0201_0603Metric -> Capacitor_SMD:C_0402_1005Metric_Pad0.74x0.62mm_HandSolder
- C3: renamed from C1; footprint Capacitor_SMD:C_0805_2012Metric -> Capacitor_SMD:C_0402_1005Metric_Pad0.74x0.62mm_HandSolder
- C30: renamed from C32; footprint Capacitor_SMD:C_0201_0603Metric -> Capacitor_SMD:C_0402_1005Metric_Pad0.74x0.62mm_HandSolder
- C31: renamed from C33; footprint Capacitor_SMD:C_0201_0603Metric -> Capacitor_SMD:C_0402_1005Metric_Pad0.74x0.62mm_HandSolder
- C33: renamed from C35; footprint Capacitor_SMD:C_1206_3216Metric -> Capacitor_SMD:C_0402_1005Metric_Pad0.74x0.62mm_HandSolder
- C34: renamed from C36; footprint Capacitor_SMD:C_1206_3216Metric -> Capacitor_SMD:C_0402_1005Metric_Pad0.74x0.62mm_HandSolder
- C37: renamed from C39; footprint Capacitor_SMD:C_0201_0603Metric -> Capacitor_SMD:C_0402_1005Metric_Pad0.74x0.62mm_HandSolder
- C39: renamed from C41; footprint Capacitor_SMD:C_1206_3216Metric -> Capacitor_SMD:C_0805_2012Metric
- C4: renamed from C3; footprint Capacitor_SMD:C_0805_2012Metric -> Capacitor_SMD:C_0402_1005Metric_Pad0.74x0.62mm_HandSolder
- C41: renamed from C43; footprint Capacitor_SMD:C_1206_3216Metric -> Capacitor_SMD:C_0805_2012Metric
- C42: renamed from C44; footprint Capacitor_SMD:C_0201_0603Metric -> Capacitor_SMD:C_0402_1005Metric_Pad0.74x0.62mm_HandSolder
- C9: renamed from C11; footprint Capacitor_SMD:C_0201_0603Metric -> Capacitor_SMD:C_0402_1005Metric_Pad0.74x0.62mm_HandSolder
- J1, J2: footprint (none) -> MicromouseHuellas:ENCODER_PAD_PADRE
- J4: renamed from J3; footprint (none) -> MicromouseHuellas:IR_SENSOR_2
- J5: renamed from J4; footprint (none) -> MicromouseHuellas:IR_SENSOR_2
- J7: renamed from J6; footprint (none) -> MicromouseHuellas:IR_SENSOR_2
- J8: renamed from J7; footprint (none) -> MicromouseHuellas:IR_SENSOR_2
- J9: renamed from J8; footprint B2B-PH-SM4-TB_LF__SN:B2B-PH-SM4-TB_LF__SN_ -> Connector_PinHeader_2.54mm:PinHeader_1x02_P2.54mm_Vertical_SMD_Pin1Left
- R10: footprint Resistor_SMD:R_0402_1005Metric_Pad0.72x0.64mm_HandSolder -> Resistor_SMD:R_0805_2012Metric
- R16: value 1K -> 330
- R18, R22, R6: footprint Resistor_SMD:R_0201_0603Metric -> Resistor_SMD:R_0402_1005Metric_Pad0.72x0.64mm_HandSolder
- R19: value 82 -> 330; footprint Resistor_SMD:R_0201_0603Metric -> Resistor_SMD:R_0402_1005Metric_Pad0.72x0.64mm_HandSolder
- R20: value 10 -> 330; footprint Resistor_SMD:R_0201_0603Metric -> Resistor_SMD:R_0402_1005Metric_Pad0.72x0.64mm_HandSolder
- R21: value 22 -> 330; footprint Resistor_SMD:R_0201_0603Metric -> Resistor_SMD:R_0402_1005Metric_Pad0.72x0.64mm_HandSolder
- R4: footprint Resistor_SMD:R_0201_0603Metric -> Resistor_SMD:R_0805_2012Metric
- renumbered C5 to C1, C13 to C11, C15 to C13, C17 to C15, C20 to C18, C21 to C19, C6 to C2, C24 to C22, C29 to C26, C30 to C28, C34 to C32, C37 to C35, C38 to C36, C40 to C38, C42 to C40, C7 to C5, C8 to C6, C2 to C7, C4 to C8, J5 to J6, IC1 to U3
Connections:
- net +3V3 is gone; now on net +3V0: R16.1
- net +3V0: no longer C27.1, C31.1, FB1.2, U1.13 (VDDA)
- net GND: now also S2.2
- net LED_10: now also U1.4 (PC15); no longer U1.61 (PB8)
- net LED_6: now also U1.61 (PB8); no longer U1.4 (PC15)
- net LED_7: now also U1.62 (PB9); no longer U1.3 (PC14)
- net LED_9: now also U1.3 (PC14); no longer U1.62 (PB9)
- net MENU_ESTADO: now also S3.1, S4.1, S5.1
- net NRST: now also S2.1
- net POW_IN: now also J3.2
- net RCC_OSC_IN: now also C23.1, Y1.3; no longer C12.1, U1.6 (PH1), Y1.1
- net RCC_OSC_OUT: now also C12.1, U1.6 (PH1), Y1.1; no longer C23.1, Y1.3
- net at R28.2: now also S3.2
- net at D2.A, Q2.3 (D): now also J3.1
- net at R29.2: now also S4.2
- net at C38.2, D10.C, U2.6 (SW): now also L1.1
- net at C39.1, R22.2: now also L1.2
- net at R30.2: now also S5.2
- new net: J3.S1 (SHIELD), J3.S2 (SHIELD)
- new net VDDA: C27.1, C31.1, FB1.2, U1.13 (VDDA)
- no-connect marks 12 -> 13
Other:
- moved on the sheet: C1, C2, C31, C5, C6, C7, C8, R2, R3

Commit message: Red 3V0 cambiada a 3V3
Parts:
- U3: value ME6211C30M5G -> ME6211C33M5G
Connections:
- net +3V0 renamed +3V3
Changed lines of the file:
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@@
 			)
 		)
-		(property "Value" "+3V0"
+		(property "Value" "+3V3"
 			(at 260.604 256.667 0)
 			(effects
@@
 			)
 		)
-		(property "Value" "+3V0"
+		(property "Value" "+3V3"
 			(at 267.97 14.732 0)
 			(effects
@@
 			)
 		)
-		(property "Value" "+3V0"
+		(property "Value" "+3V3"
 			(at 274.32 256.921 0)
 			(effects
@@
 			)
 		)
-		(property "Value" "+3V0"
+		(property "Value" "+3V3"
 			(at 288.036 256.921 0)
 			(effects
@@
 			)
 		)
-		(property "Value" "+3V0"
+		(property "Value" "+3V3"
 			(at 246.38 256.667 0)
 			(effects
@@
 			)
 		)
-		(property "Value" "+3V0"
+		(property "Value" "+3V3"
 			(at 226.06 74.93 0)
 			(effects
@@
 			)
 		)
-		(property "Value" "+3V0"
+		(property "Value" "+3V3"
 			(at 400.304 204.47 0)
 			(effects
@@
 			)
 		)
-		(property "Value" "+3V0"
+		(property "Value" "+3V3"
 			(at 113.03 59.944 0)
 			(effects
@@
 			)
 		)
-		(property "Value" "+3V0"
+		(property "Value" "+3V3"
 			(at 217.424 261.366 0)
 			(effects
@@
 			)
 		)
-		(property "Value" "+3V0"
+		(property "Value" "+3V3"
 			(at 384.556 88.138 0)
 			(effects
@@
 			)
 		)
-		(property "Value" "+3V0"
+		(property "Value" "+3V3"
 			(at 337.82 202.184 0)
 			(effects
@@
 			)
 		)
-		(property "Value" "+3V0"
+		(property "Value" "+3V3"
 			(at 308.229 165.1 0)
 			(effects
@@
 			)
 		)
-		(property "Value" "+3V0"
+		(property "Value" "+3V3"
 			(at 232.156 261.366 0)
 			(effects
@@
 			)
 		)
-		(property "Value" "ME6211C30M5G"
+		(property "Value" "ME6211C33M5G"
 			(at 363.22 85.09 0)
 			(effects
@@
 			)
 		)
-		(property "Value" "+3V0"
+		(property "Value" "+3V3"
 			(at 226.568 161.544 0)
 			(effects
@@
 			)
 		)
-		(property "Value" "+3V0"
+		(property "Value" "+3V3"
 			(at 72.898 84.836 0)
 			(effects
@@
 			)
 		)
-		(property "Value" "+3V0"
+		(property "Value" "+3V3"
 			(at 58.42 84.328 0)
 			(effects
@@
 			)
 		)
-		(property "Value" "+3V0"
+		(property "Value" "+3V3"
 			(at 105.918 59.69 0)
 			(effects

Commit message: Modelos 3D agregados
Other:
- removed sheet AS5048_Der
- removed sheet AS5048_Izq
Changed lines of the file:
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@@
-	)
-	(sheet
-		(at 188.722 106.934)
-		(size 16.51 15.24)
-		(exclude_from_sim no)
-		(in_bom yes)
-		(on_board yes)
-		(dnp no)
-		(stroke
-			(width 0.1524)
-			(type solid)
-		)
-		(fill
-			(color 0 0 0 0.0000)
-		)
-		(property "Sheetname" "AS5048_Izq"
-			(at 188.722 106.2224 0)
-			(effects
-				(font
-					(size 1.27 1.27)
-				)
-				(justify left bottom)
-			)
-		)
-		(property "Sheetfile" "AS5048_Izq.kicad_sch"
-			(at 182.372 122.936 0)
-			(effects
-				(font
-					(size 1.27 1.27)
-				)
-				(justify left top)
-			)
-		)
-		(instances
-			(project "Micromouse"
-				(path "/96b72c82-8e98-4b00-820e-849de0fa96c7"
-					(page "2")
-				)
-			)
-		)
-	)
-	(sheet
-		(at 188.976 130.048)
-		(size 16.51 15.24)
-		(exclude_from_sim no)
-		(in_bom yes)
-		(on_board yes)
-		(dnp no)
-		(stroke
-			(width 0.1524)
-			(type solid)
-		)
-		(fill
-			(color 0 0 0 0.0000)
-		)
-		(property "Sheetname" "AS5048_Der"
-			(at 188.976 129.3364 0)
-			(effects
-				(font
-					(size 1.27 1.27)
-				)
-				(justify left bottom)
-			)
-		)
-		(property "Sheetfile" "AS5048_Der.kicad_sch"
-			(at 183.388 146.431 0)
-			(effects
-				(font
-					(size 1.27 1.27)
-				)
-				(justify left top)
-			)
-		)
-		(instances
-			(project "Micromouse"
-				(path "/96b72c82-8e98-4b00-820e-849de0fa96c7"
-					(page "3")
-				)
-			)
-		)
 	)
 	(sheet
@@
 	)
 	(sheet
-		(at 188.976 155.956)
+		(at 153.416 183.642)
 		(size 16.51 15.24)
 		(exclude_from_sim no)
@@
 		)
 		(property "Sheetname" "IR_sensor"
-			(at 188.976 155.2444 0)
+			(at 153.416 182.9304 0)
 			(effects
 				(font
@@
 		)
 		(property "Sheetfile" "IR_sensor.kicad_sch"
-			(at 184.404 171.958 0)
+			(at 148.844 199.644 0)
 			(effects
 				(font
