File: Micromouse/PCB_Files/Micromouse.kicad_sch (KiCad schematic)
At the start: 114 parts, among them J1 AS5048_Izq, J2 AS5048_Der, J3 MOT_FAN, J4 IR_LAT_Der, J5 IR_LAT_Izq, J6 ST_LINK, J7 IR_FRONT_Der, J8 IR_FRONT_Izq, J9 Lipo, Q1 AO3400A, Q2 AO3400A, Q3 AON7423, U1 STM32F405RGTx, U2 MP2359DJ-LF-Z, U3 ME6211C33M5G, Y1 8MHz

Commit message: Fe de erratas en circuito de potencia micromouse
Other:
- note added: "1"
- note added: "2"
- note added: "3"
- note added: "4"
- note added: "Fe de erratas: 1. Puentear +3V3 con +3V3(ST-LINK) 2. Puentear el pin 2 del inductor con +5V 3. Usar un inductor de 3.3uH 4. Añadir capacitor de 10uF entre IN y GND 5. Modificar físicamente la PCB para que el pin 2 del switch sólo esté conectado a GND y viceversa"
Changed lines of the file:
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@@
 		)
 	)
+	(text "Fe de erratas:\n\n1. Puentear +3V3 con +3V3(ST-LINK)\n2. Puentear el pin 2 del inductor con +5V\n3. Usar un inductor de 3.3uH\n4. Añadir capacitor de 10uF entre IN y GND\n5. Modificar físicamente la PCB para que el\n   pin 2 del switch sólo esté conectado a\n   GND y viceversa"
+		(exclude_from_sim no)
+		(at 431.8 22.352 0)
+		(effects
+			(font
+				(size 5 5)
+			)
+			(justify left)
+		)
+	)
 	(text "Pads de conexión\n"
 		(exclude_from_sim no)
@@
 		)
 	)
+	(text "2"
+		(exclude_from_sim no)
+		(at 390.906 57.404 0)
+		(effects
+			(font
+				(size 1.27 1.27)
+			)
+			(justify left)
+		)
+	)
 	(text "Botón NRST"
 		(exclude_from_sim no)
@@
 		)
 	)
+	(text "3"
+		(exclude_from_sim no)
+		(at 387.858 33.782 0)
+		(effects
+			(font
+				(size 1.27 1.27)
+			)
+			(justify left)
+		)
+	)
+	(text "4"
+		(exclude_from_sim no)
+		(at 321.564 27.178 0)
+		(effects
+			(font
+				(size 1.27 1.27)
+			)
+			(justify left)
+		)
+	)
+	(text "1"
+		(exclude_from_sim no)
+		(at 403.098 99.06 0)
+		(effects
+			(font
+				(size 1.27 1.27)
+			)
+			(justify left)
+		)
+	)
 	(text "Circuito del reloj"
 		(exclude_from_sim no)
@@
 		)
 	)
+	(polyline
+		(pts
+			(xy 377.952 34.036) (xy 377.952 56.642)
+		)
+		(stroke
+			(width 0)
+			(type dash_dot)
+		)
+	)
 	(wire
 		(pts
@@
 		)
 	)
+	(polyline
+		(pts
+			(xy 379.476 57.404) (xy 379.476 64.262)
+		)
+		(stroke
+			(width 0)
+			(type dash_dot)
+		)
+	)
 	(wire
 		(pts
@@
 		)
 	)
+	(polyline
+		(pts
+			(xy 379.476 57.404) (xy 390.398 57.404)
+		)
+		(stroke
+			(width 0)
+			(type dash_dot)
+		)
+	)
 	(wire
 		(pts
@@
 		)
 	)
+	(polyline
+		(pts
+			(xy 390.398 64.262) (xy 379.476 64.262)
+		)
+		(stroke
+			(width 0)
+			(type dash_dot)
+		)
+	)
 	(wire
 		(pts
@@
 		)
 	)
+	(polyline
+		(pts
+			(xy 308.864 84.582) (xy 308.864 68.072)
+		)
+		(stroke
+			(width 0)
+			(type dash_dot)
+		)
+	)
 	(wire
 		(pts
@@
 		)
 	)
+	(polyline
+		(pts
+			(xy 390.398 57.404) (xy 390.398 64.262)
+		)
+		(stroke
+			(width 0)
+			(type dash_dot)
+		)
+	)
 	(wire
 		(pts
@@
 		)
 	)
+	(polyline
+		(pts
+			(xy 306.832 27.686) (xy 306.832 36.576)
+		)
+		(stroke
+			(width 0)
+			(type dash_dot)
+		)
+	)
 	(wire
 		(pts
@@
 		)
 	)
+	(polyline
+		(pts
+			(xy 387.604 56.642) (xy 377.952 56.642)
+		)
+		(stroke
+			(width 0)
+			(type dash_dot)
+		)
+	)
 	(wire
 		(pts
@@
 		)
 	)
+	(polyline
+		(pts
+			(xy 294.132 84.582) (xy 308.864 84.582)
+		)
+		(stroke
+			(width 0)
+			(type dash_dot)
+		)
+	)
 	(wire
 		(pts
@@
 		)
 	)
+	(polyline
+		(pts
+			(xy 377.952 34.036) (xy 387.604 34.036)
+		)
+		(stroke
+			(width 0)
+			(type dash_dot)
+		)
+	)
 	(wire
 		(pts
@@
 		)
 	)
+	(polyline
+		(pts
+			(xy 321.31 36.576) (xy 306.832 36.576)
+		)
+		(stroke
+			(width 0)
+			(type dash_dot)
+		)
+	)
 	(wire
 		(pts
@@
 		)
 	)
+	(polyline
+		(pts
+			(xy 387.604 34.036) (xy 387.604 56.642)
+		)
+		(stroke
+			(width 0)
+			(type dash_dot)
+		)
+	)
 	(wire
 		(pts
@@
 		)
 	)
+	(polyline
+		(pts
+			(xy 387.858 88.646) (xy 402.336 88.646)
+		)
+		(stroke
+			(width 0)
+			(type dash_dot)
+		)
+	)
 	(wire
 		(pts
@@
 		)
 	)
+	(polyline
+		(pts
+			(xy 387.858 97.79) (xy 402.336 97.79)
+		)
+		(stroke
+			(width 0)
+			(type dash_dot)
+		)
+	)
 	(wire
 		(pts
@@
 		)
 	)
+	(polyline
+		(pts
+			(xy 294.132 68.072) (xy 308.864 68.072)
+		)
+		(stroke
+			(width 0)
+			(type dash_dot)
+		)
+	)
 	(wire
 		(pts
@@
 		)
 	)
+	(polyline
+		(pts
+			(xy 402.336 88.646) (xy 402.336 97.79)
+		)
+		(stroke
+			(width 0)
+			(type dash_dot)
+		)
+	)
 	(wire
 		(pts
@@
 		)
 	)
+	(polyline
+		(pts
+			(xy 306.832 27.686) (xy 321.31 27.686)
+		)
+		(stroke
+			(width 0)
+			(type dash_dot)
+		)
+	)
 	(wire
 		(pts
@@
 		)
 	)
+	(polyline
+		(pts
+			(xy 294.132 68.072) (xy 294.132 84.582)
+		)
+		(stroke
+			(width 0)
+			(type dash_dot)
+		)
+	)
 	(wire
 		(pts
@@
 		)
 	)
+	(polyline
+		(pts
+			(xy 321.31 27.686) (xy 321.31 36.576)
+		)
+		(stroke
+			(width 0)
+			(type dash_dot)
+		)
+	)
 	(wire
 		(pts
@@
 		)
 	)
+	(polyline
+		(pts
+			(xy 387.858 88.646) (xy 387.858 97.79)
+		)
+		(stroke
+			(width 0)
+			(type dash_dot)
+		)
+	)
